File: Cloud-Star-Lights-PCB/Cloud-Star-Lights-PCB.kicad_sch (KiCad schematic)
At the start: 170 parts, among them J1 Conn_01x02, J10 Conn_01x02, J11 Conn_01x02, J12 Conn_01x02, J13 Conn_01x02, J14 Conn_01x02, J15 Conn_01x02, J16 Conn_01x02, J17 Conn_01x02, J18 Conn_01x02, J19 Conn_01x02, J2 Conn_01x02, J20 Conn_01x02, J21 Conn_01x02, J22 Conn_01x02, J23 Conn_01x02, J24 Conn_01x02, J25 Conn_01x02, J26 Conn_01x02, J27 Conn_01x02, J28 Conn_01x02, J29 Conn_01x02, J3 Conn_01x02, J30 Conn_01x02, J31 Conn_01x04, J32 Conn_01x04, J33 Conn_01x04, J34 Conn_01x04, J35 Conn_01x04, J36 Conn_01x04, J37 Conn_01x04, J38 Conn_01x04, J39 Conn_01x04, J4 Conn_01x02, J40 Conn_01x04, J41 Conn_01x04, J42 Conn_01x04, J43 Conn_01x04, J44 Conn_01x04, J45 Conn_01x04, J46 Conn_01x02, J47 Conn_01x02, J48 Conn_01x02, J49 Conn_01x03, J5 Conn_01x02, J50 Conn_01x02, J6 Conn_01x02, J7 Conn_01x02, J8 Conn_01x02, J9 Conn_01x02, Q1 2N3906, Q10 2N3906, Q11 2N3906, Q12 2N3906, Q13 2N3906, Q14 2N3906, Q15 2N3906, Q16 2N3906, Q17 2N3906, Q18 2N3906, Q19 2N3906, Q2 2N3906, Q20 2N3906, Q21 2N3906, Q22 2N3906, Q23 2N3906, Q24 2N3906, Q25 2N3906, Q26 2N3906, Q27 2N3906, Q28 2N3906, Q29 2N3906, Q3 2N3906, Q30 2N3906, Q31 2N3906, Q32 2N3906, Q33 2N3906, Q34 2N3906, Q35 2N3906, Q36 2N3906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

Commit message: Change a connector to a screw terminal
Parts:
- removed J48: Conn_01x02, Library:MAX_MX126-5.0-02P-GN01-Cu-S-A, symbol Connector_Generic:Conn_01x02
- added J48: Screw_Terminal_01x02, symbol Connector:Screw_Terminal_01x02
Connections:
- net +5V: now also J48.1 (Pin_1)
- net GND: now also J48.2 (Pin_2)
Changed lines of the file:
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@@
+    )
+  )
+  (symbol (lib_id "Connector:Screw_Terminal_01x02") (at 421.64 177.8 0) (unit 1)
+    (in_bom yes) (on_board yes) (dnp no) (fields_autoplaced)
+    (property "Reference" "J48" (at 424.18 179.07 0)
+      (effects (font (size 1.27 1.27)) (justify left))
+    )
+    (property "Value" "Screw_Terminal_01x02" (at 424.18 180.34 0)
+      (effects (font (size 1.27 1.27)) (justify left) hide)
+    )
+    (property "Footprint" "" (at 421.64 177.8 0)
+      (effects (font (size 1.27 1.27)) hide)
+    )
+    (property "Datasheet" "~" (at 421.64 177.8 0)
+      (effects (font (size 1.27 1.27)) hide)
+    )
+    (pin "1")
+    (pin "2")
+    (instances
+      (project "Cloud-Star-Lights-PCB"
+        (path "/6eaa0fe7-97a1-430a-b476-3854a870e462"
+          (reference "J48") (unit 1)
+        )
+      )
     )
   )
@@
         )
       )
-    )
-  )
-  (symbol (lib_id "Connector_Generic:Conn_01x02") (at 421.64 177.8 0) (unit 1)
-    (in_bom yes) (on_board yes) (dnp no) (fields_autoplaced)
-    (property "Reference" "J48" (at 424.18 179.07 0)
-      (effects (font (size 1.27 1.27)) (justify left))
-    )
-    (property "Value" "Conn_01x02" (at 424.18 180.34 0)
-      (effects (font (size 1.27 1.27)) (justify left) hide)
-    )
-    (property "Footprint" "Library:MAX_MX126-5.0-02P-GN01-Cu-S-A" (at 421.64 177.8 0)
-      (effects (font (size 1.27 1.27)) hide)
-    )
-    (property "Datasheet" "~" (at 421.64 177.8 0)
-      (effects (font (size 1.27 1.27)) hide)
-    )
-    (pin "1")
-    (pin "2")
-    (instances
-      (project "Cloud-Star-Lights-PCB"
-        (path "/6eaa0fe7-97a1-430a-b476-3854a870e462"
-          (reference "J48") (unit 1)
-        )
-      )
