File: Cloud-Star-Lights-PCB/Cloud-Star-Lights-PCB.kicad_sch (KiCad schematic)
At the start: 159 parts, among them J1 Conn_01x02, J10 Conn_01x02, J11 Conn_01x02, J12 Conn_01x02, J13 Conn_01x02, J14 Conn_01x02, J15 Conn_01x02, J16 Conn_01x02, J17 Conn_01x02, J18 Conn_01x02, J19 Conn_01x02, J2 Conn_01x02, J20 Conn_01x02, J21 Conn_01x02, J22 Conn_01x02, J23 Conn_01x02, J24 Conn_01x02, J25 Conn_01x02, J26 Conn_01x02, J27 Conn_01x02, J28 Conn_01x02, J29 Conn_01x02, J3 Conn_01x02, J30 Conn_01x02, J31 Conn_01x04, J32 Conn_01x04, J33 Conn_01x04, J34 Conn_01x04, J35 Conn_01x04, J36 Conn_01x04, J37 Conn_01x04, J38 Conn_01x04, J39 Conn_01x04, J4 Conn_01x02, J40 Conn_01x04, J41 Conn_01x04, J42 Conn_01x04, J43 Conn_01x04, J44 Conn_01x04, J45 Conn_01x04, J46 Conn_01x02, J47 Conn_01x02, J48 Conn_01x02, J49 Conn_01x03, J5 Conn_01x02, J6 Conn_01x02, J7 Conn_01x02, J8 Conn_01x02, J9 Conn_01x02, Q1 2N3906, Q10 2N3906, Q11 2N3906, Q12 2N3906, Q13 2N3906, Q14 2N3906, Q15 2N3906, Q16 2N3906, Q17 2N3906, Q18 2N3906, Q19 2N3906, Q2 2N3906, Q20 2N3906, Q21 2N3906, Q22 2N3906, Q23 2N3906, Q24 2N3906, Q25 2N3906, Q26 2N3906, Q27 2N3906, Q28 2N3906, Q29 2N3906, Q3 2N3906, Q30 2N3906, Q4 2N3906, Q5 2N3906, Q6 2N3906, Q7 2N3906, Q8 2N3906, Q9 2N3906, U1 PCA9685 Breakout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

Commit message: Schematic
Parts:
- removed Q31, Q32, Q33, Q34, Q35, Q36, Q37, Q38, Q39, Q40, Q41, Q42, Q43, Q44, Q45, Q46, Q47, Q48, Q49, Q50, Q51, Q52, Q53, Q54, Q55, Q56, Q57, Q58, Q59, Q60, Q61, Q62, Q63, Q64, Q65, Q66, Q67, Q68, Q69, Q70, Q71, Q72, Q73, Q74, Q75: ~, Library:AP5N10S, symbol Library:AP5N10S
- removed U1, U3, U4: PCA9685 Breakout, symbol Library:PCA9685_Breakout
- added C1, C2, C4: 10uf, Capacitor_SMD:C_0201_0603Metric_Pad0.64x0.40mm_HandSolder, symbol Device:C
- added C5, C6: 0.1uF, Capacitor_SMD:C_0201_0603Metric_Pad0.64x0.40mm_HandSolder, symbol Device:C
- added J50: Conn_01x02, Library:MAX_MX126-5.0-02P-GN01-Cu-S-A, symbol Connector_Generic:Conn_01x02
- added Q31, Q32, Q33, Q34, Q35, Q36, Q37, Q38, Q39, Q40, Q41, Q42, Q43, Q44, Q45, Q46, Q47, Q48, Q49, Q50, Q51, Q52, Q53, Q54, Q55, Q56, Q57, Q58, Q59, Q60, Q61, Q62, Q63, Q64, Q65, Q66, Q67, Q68, Q69, Q70, Q71, Q72, Q73, Q74, Q75: 2N3906, Package_TO_SOT_THT:TO-92_Inline, symbol Transistor_BJT:2N3906
- added R31, R32, R33, R34, R35: 10kΩ, Resistor_SMD:R_0201_0603Metric_Pad0.64x0.40mm_HandSolder, symbol Device:R
- added U1, U3, U4: PCA9635, Package_SO:TSSOP-28_4.4x9.7mm_P0.65mm, symbol Driver_LED:PCA9635
- C3: renamed from C1; footprint (none) -> Capacitor_SMD:C_0201_0603Metric_Pad0.64x0.40mm_HandSolder
- J1, J10, J11, J12, J13, J14, J15, J16, J17, J18, J19, J2, J20, J21, J22, J23, J24, J25, J26, J27, J28, J29, J3, J30, J4, J46, J47, J48, J5, J6, J7, J8, J9: footprint (none) -> Library:MAX_MX126-5.0-02P-GN01-Cu-S-A
- J31, J32, J33, J34, J35, J36, J37, J38, J39, J40, J41, J42, J43, J44, J45: footprint (none) -> Library:JILN_JL301-50004U01
- J49: footprint (none) -> Library:Cixi_Kefa_Elec_KF135T-10.16-3P
Connections:
- net +3.3V: now also J47.1 (Pin_1), C1.2, C2.2, C4.2, C5.2, R32.1, R33.1, U1.2 (A1), U1.24 (A5), U1.25 (A6), U1.28 (VDD), U1.3 (A2), U1.4 (A3), U1.5 (A4), U3.2 (A1), U3.24 (A5), U3.25 (A6), U3.28 (VDD), U3.3 (A2), U3.4 (A3), U3.5 (A4), U4.2 (A1), U4.24 (A5), U4.25 (A6), U4.28 (VDD), U4.3 (A2), U4.4 (A3), U4.5 (A4); no longer J48.1 (Pin_1)
- net +5V: now also J48.1 (Pin_1), R1.1, R10.1, R11.1, R12.1, R13.1, R14.1, R15.1, R16.1, R17.1, R18.1, R19.1, R2.1, R20.1, R21.1, R22.1, R23.1, R24.1, R25.1, R26.1, R27.1, R28.1, R29.1, R3.1, R30.1, R4.1, R5.1, R6.1, R7.1, R8.1, R9.1, C6.2; no longer Q1.1 (E), Q10.1 (E), Q11.1 (E), Q12.1 (E), Q13.1 (E), Q14.1 (E), Q15.1 (E), Q16.1 (E), Q17.1 (E), Q18.1 (E), Q19.1 (E), Q2.1 (E), Q20.1 (E), Q21.1 (E), Q22.1 (E), Q23.1 (E), Q24.1 (E), Q25.1 (E), Q27.1 (E), Q28.1 (E), Q29.1 (E), Q3.1 (E), Q30.1 (E), Q4.1 (E), Q5.1 (E), Q6.1 (E), Q7.1 (E), Q8.1 (E), Q9.1 (E)
- net Cloud_Control_B1: now also Q42.2 (B), Q57.2 (B), Q72.2 (B), U4.17 (LED10)
- net Cloud_Control_B2: now also Q43.2 (B), Q58.2 (B), Q73.2 (B), U4.18 (LED11)
- net Cloud_Control_B3: now also Q44.2 (B), Q59.2 (B), Q74.2 (B), U4.19 (LED12)
- net Cloud_Control_B4: now also Q45.2 (B), Q60.2 (B), Q75.2 (B), U4.20 (LED13)
- net Cloud_Control_B5: now also Q41.2 (B), Q56.2 (B), Q71.2 (B), U4.21 (LED14)
- net Cloud_Control_G1: now also Q37.2 (B), Q52.2 (B), Q67.2 (B), U4.11 (LED5)
- net Cloud_Control_G2: now also Q38.2 (B), Q53.2 (B), Q68.2 (B), U4.12 (LED6)
- net Cloud_Control_G3: now also Q39.2 (B), Q54.2 (B), Q69.2 (B), U4.13 (LED7)
- net Cloud_Control_G4: now also Q40.2 (B), Q55.2 (B), Q70.2 (B), U4.15 (LED8)
- net Cloud_Control_G5: now also Q36.2 (B), Q51.2 (B), Q66.2 (B), U4.16 (LED9)
- net Cloud_Control_R1: now also Q32.2 (B), Q47.2 (B), Q62.2 (B), U4.6 (LED0)
- net Cloud_Control_R2: now also Q33.2 (B), Q48.2 (B), Q63.2 (B), U4.7 (LED1)
- net Cloud_Control_R3: now also Q34.2 (B), Q49.2 (B), Q64.2 (B), U4.8 (LED2)
- net Cloud_Control_R4: now also Q35.2 (B), Q50.2 (B), Q65.2 (B), U4.9 (LED3)
- net Cloud_Control_R5: now also Q31.2 (B), Q46.2 (B), Q61.2 (B), U4.10 (LED4)
- net GND: now also Q1.3 (C), Q10.3 (C), Q11.3 (C), Q12.3 (C), Q13.3 (C), Q14.3 (C), Q15.3 (C), Q16.3 (C), Q17.3 (C), Q18.3 (C), Q19.3 (C), Q2.3 (C), Q20.3 (C), Q21.3 (C), Q22.3 (C), Q23.3 (C), Q24.3 (C), Q25.3 (C), Q26.3 (C), Q27.3 (C), Q28.3 (C), Q29.3 (C), Q3.3 (C), Q30.3 (C), Q4.3 (C), Q5.3 (C), Q6.3 (C), Q7.3 (C), Q8.3 (C), Q9.3 (C), C1.1, C2.1, C4.1, C5.1, C6.1, Q31.3 (C), Q32.3 (C), Q33.3 (C), Q34.3 (C), Q35.3 (C), Q36.3 (C), Q37.3 (C), Q38.3 (C), Q39.3 (C), Q40.3 (C), Q41.3 (C), Q42.3 (C), Q43.3 (C), Q44.3 (C), Q45.3 (C), Q46.3 (C), Q47.3 (C), Q48.3 (C), Q49.3 (C), Q50.3 (C), Q51.3 (C), Q52.3 (C), Q53.3 (C), Q54.3 (C), Q55.3 (C), Q56.3 (C), Q57.3 (C), Q58.3 (C), Q59.3 (C), Q60.3 (C), Q61.3 (C), Q62.3 (C), Q63.3 (C), Q64.3 (C), Q65.3 (C), Q66.3 (C), Q67.3 (C), Q68.3 (C), Q69.3 (C), Q70.3 (C), Q71.3 (C), Q72.3 (C), Q73.3 (C), Q74.3 (C), Q75.3 (C), R31.2, R34.2, R35.2, U1.1 (A0), U1.14 (VSS), U3.1 (A0), U3.14 (VSS), U4.1 (A0), U4.14 (VSS); no longer J1.2 (Pin_2), J10.2 (Pin_2), J11.2 (Pin_2), J12.2 (Pin_2), J13.2 (Pin_2), J14.2 (Pin_2), J15.2 (Pin_2), J16.2 (Pin_2), J17.2 (Pin_2), J18.2 (Pin_2), J19.2 (Pin_2), J2.2 (Pin_2), J20.2 (Pin_2), J21.2 (Pin_2), J22.2 (Pin_2), J23.2 (Pin_2), J24.2 (Pin_2), J25.2 (Pin_2), J26.2 (Pin_2), J27.2 (Pin_2), J28.2 (Pin_2), J29.2 (Pin_2), J3.2 (Pin_2), J30.2 (Pin_2), J4.2 (Pin_2), J47.1 (Pin_1), J5.2 (Pin_2), J6.2 (Pin_2), J7.2 (Pin_2), J8.2 (Pin_2), J9.2 (Pin_2)
- net SCL: now also R32.2, U1.26 (SCL), U3.26 (SCL), U4.26 (SCL)
- net SDA: now also R33.2, U1.27 (SDA), U3.27 (SDA), U4.27 (SDA)
- net Star_Control_1: now also U1.6 (LED0)
- net Star_Control_10: now also U1.16 (LED9)
- net Star_Control_11: now also U1.17 (LED10)
- net Star_Control_12: now also U1.18 (LED11)
- net Star_Control_13: now also U1.19 (LED12)
- net Star_Control_14: now also U1.20 (LED13)
- net Star_Control_15: now also U1.21 (LED14)
- net Star_Control_16: now also U3.6 (LED0)
- net Star_Control_17: now also U3.7 (LED1)
- net Star_Control_18: now also U3.8 (LED2)
- net Star_Control_19: now also U3.9 (LED3)
- net Star_Control_2: now also U1.7 (LED1)
- net Star_Control_20: now also U3.10 (LED4)
- net Star_Control_21: now also U3.11 (LED5)
- net Star_Control_22: now also U3.12 (LED6)
- net Star_Control_23: now also U3.13 (LED7)
- net Star_Control_24: now also U3.15 (LED8)
- net Star_Control_25: now also U3.16 (LED9)
- net Star_Control_26: now also U3.17 (LED10)
- net Star_Control_27: now also U3.18 (LED11)
- net Star_Control_28: now also U3.19 (LED12)
- net Star_Control_29: now also U3.20 (LED13)
- net Star_Control_3: now also U1.8 (LED2)
- net Star_Control_30: now also U3.21 (LED14)
- net Star_Control_4: now also U1.9 (LED3)
- net Star_Control_5: now also U1.10 (LED4)
- net Star_Control_6: now also U1.11 (LED5)
- net Star_Control_7: now also U1.12 (LED6)
- net Star_Control_8: now also U1.13 (LED7)
- net Star_Control_9: now also U1.15 (LED8)
- net at J43.3 (Pin_3): now also Q73.1 (E)
- net at J35.1 (Pin_1): now also Q35.1 (E)
- net at J35.3 (Pin_3): now also Q45.1 (E)
- net at J31.1 (Pin_1): now also Q31.1 (E)
- net at J31.2 (Pin_2): now also Q36.1 (E)
- net at J31.3 (Pin_3): now also Q41.1 (E)
- net at J36.1 (Pin_1): now also Q46.1 (E)
- net at J36.2 (Pin_2): now also Q51.1 (E)
- net at J36.3 (Pin_3): now also Q56.1 (E)
- net at J42.2 (Pin_2): now also Q67.1 (E)
- net at J42.1 (Pin_1): now also Q62.1 (E)
- net at J42.3 (Pin_3): now also Q72.1 (E)
- net at J33.1 (Pin_1): now also Q33.1 (E)
- net at J32.1 (Pin_1): now also Q32.1 (E)
- net at J35.2 (Pin_2): now also Q40.1 (E)
- net at J45.1 (Pin_1): now also Q65.1 (E)
- net at J45.2 (Pin_2): now also Q70.1 (E)
- net at J45.3 (Pin_3): now also Q75.1 (E)
- net at J40.2 (Pin_2): now also Q55.1 (E)
- net at J41.2 (Pin_2): now also Q66.1 (E)
- net at J38.1 (Pin_1): now also Q48.1 (E)
- net at J32.3 (Pin_3): now also Q42.1 (E)
- net at J44.2 (Pin_2): now also Q69.1 (E)
- net at J37.2 (Pin_2): now also Q52.1 (E)
- net at J44.1 (Pin_1): now also Q64.1 (E)
- net at J44.3 (Pin_3): now also Q74.1 (E)
- net at J37.3 (Pin_3): now also Q57.1 (E)
- net at J34.1 (Pin_1): now also Q34.1 (E)
- net at J34.2 (Pin_2): now also Q39.1 (E)
- net at J34.3 (Pin_3): now also Q44.1 (E)
- net at J39.2 (Pin_2): now also Q54.1 (E)
- net at J33.3 (Pin_3): now also Q43.1 (E)
- net at J38.2 (Pin_2): now also Q53.1 (E)
- net at J38.3 (Pin_3): now also Q58.1 (E)
- net at J41.1 (Pin_1): now also Q61.1 (E)
- net at J41.3 (Pin_3): now also Q71.1 (E)
- net at J37.1 (Pin_1): now also Q47.1 (E)
- net at J40.3 (Pin_3): now also Q60.1 (E)
- net at J32.2 (Pin_2): now also Q37.1 (E)
- net at J33.2 (Pin_2): now also Q38.1 (E)
- net at J43.1 (Pin_1): now also Q63.1 (E)
- net at J43.2 (Pin_2): now also Q68.1 (E)
- net at J39.1 (Pin_1): now also Q49.1 (E)
- net at Q26.1 (E): now also J26.2 (Pin_2)
- net at J39.3 (Pin_3): now also Q59.1 (E)
- net at J40.1 (Pin_1): now also Q50.1 (E)
- net at U2.12 (RX0/D3): now also J50.1 (Pin_1)
- net at U2.13 (TX0/D1): now also J50.2 (Pin_2)
- net OUTPUT_ENABLE: no longer names the net of U2.15 (D23/VSPI_MOSI)
- new net: J9.2 (Pin_2), Q9.1 (E)
- new net: J28.2 (Pin_2), Q28.1 (E)
- new net: J17.2 (Pin_2), Q17.1 (E)
- new net: J6.2 (Pin_2), Q6.1 (E)
- new net: J3.2 (Pin_2), Q3.1 (E)
- new net: J1.2 (Pin_2), Q1.1 (E)
- new net: R34.1, U3.23 (~{OE})
- new net: J25.2 (Pin_2), Q25.1 (E)
- new net: J29.2 (Pin_2), Q29.1 (E)
- new net: J22.2 (Pin_2), Q22.1 (E)
- new net: J10.2 (Pin_2), Q10.1 (E)
- new net: J11.2 (Pin_2), Q11.1 (E)
- new net: J15.2 (Pin_2), Q15.1 (E)
- new net: J7.2 (Pin_2), Q7.1 (E)
- new net: R31.1, U1.23 (~{OE})
- new net: J4.2 (Pin_2), Q4.1 (E)
- new net: R35.1, U4.23 (~{OE})
- new net: J20.2 (Pin_2), Q20.1 (E)
- new net: J8.2 (Pin_2), Q8.1 (E)
- new net: J16.2 (Pin_2), Q16.1 (E)
- new net: J5.2 (Pin_2), Q5.1 (E)
- new net: J2.2 (Pin_2), Q2.1 (E)
- new net: J12.2 (Pin_2), Q12.1 (E)
- new net: J14.2 (Pin_2), Q14.1 (E)
- new net: J27.2 (Pin_2), Q27.1 (E)
- new net: J19.2 (Pin_2), Q19.1 (E)
- new net: J13.2 (Pin_2), Q13.1 (E)
- new net: J23.2 (Pin_2), Q23.1 (E)
- new net: J18.2 (Pin_2), Q18.1 (E)
- new net: J24.2 (Pin_2), Q24.1 (E)
- new net: J30.2 (Pin_2), Q30.1 (E)
- new net: J21.2 (Pin_2), Q21.1 (E)
- no-connect marks 25 -> 24
Other:
- note removed: "30 LED's per meter Cut lines every 10cm 50mA/10cm -> 5mA/cm per channel Clouds have 60cm -> 300mA / 0.3A per channel 0.3A * 5v = 1.5W per LED LED lines have a common power Thus transistor on opposite side compared to the star config"
- note removed: "30 Stars 0.625W / 0.11WperLED = 5 LED max per board 3 LED's per board * 0.05A per LED = 0.15A for the board V = IR (5V - 2.15V) = 0.15A * R R = 2.85V / 0.15A R = 19ohm = 22ohm Transistor could be put on either side, I think it's cleaner being right before the resistor"
- moved on the sheet: C3, J1, J46, J47, J48, J49, R1, U2

Commit message: before I run the autoroute4
Parts:
- removed J49: Conn_01x03, Library:Cixi_Kefa_Elec_KF135T-10.16-3P, symbol Connector_Generic:Conn_01x03
- added H1, H2, H3, H4: MountingHole_Pad, MountingHole:MountingHole_4.3mm_M4_DIN965_Pad_TopBottom, symbol Mechanical:MountingHole_Pad
- added J49, J51: Screw_Terminal_01x02, TerminalBlock:TerminalBlock_bornier-2_P5.08mm, symbol Connector:Screw_Terminal_01x02
- C1, C2, C3, C4, C5, C6: footprint Capacitor_SMD:C_0201_0603Metric_Pad0.64x0.40mm_HandSolder -> Capacitor_SMD:C_1206_3216Metric_Pad1.33x1.80mm_HandSolder
- J46: footprint Library:MAX_MX126-5.0-02P-GN01-Cu-S-A -> Connector_PinHeader_2.54mm:PinHeader_1x02_P2.54mm_Vertical
- Q1, Q10, Q11, Q12, Q13, Q14, Q15, Q16, Q17, Q18, Q19, Q2, Q20, Q21, Q22, Q23, Q24, Q25, Q26, Q27, Q28, Q29, Q3, Q30, Q31, Q32, Q33, Q34, Q35, Q36, Q37, Q38, Q39, Q4, Q40, Q41, Q42, Q43, Q44, Q45, Q46, Q47, Q48, Q49, Q5, Q50, Q51, Q52, Q53, Q54, Q55, Q56, Q57, Q58, Q59, Q6, Q60, Q61, Q62, Q63, Q64, Q65, Q66, Q67, Q68, Q69, Q7, Q70, Q71, Q72, Q73, Q74, Q75, Q8, Q9: footprint Package_TO_SOT_THT:TO-92_Inline -> Package_TO_SOT_THT:TO-92S_Wide
- R1, R10, R11, R12, R13, R14, R15, R16, R17, R18, R19, R2, R20, R21, R22, R23, R24, R25, R26, R27, R28, R29, R3, R30, R31, R32, R33, R34, R35, R4, R5, R6, R7, R8, R9: footprint Resistor_SMD:R_0201_0603Metric_Pad0.64x0.40mm_HandSolder -> Resistor_SMD:R_1206_3216Metric_Pad1.30x1.75mm_HandSolder
Connections:
- net +3.3V: now also J51.1 (Pin_1)
- net +5V: now also J49.1 (Pin_1)
- net GND: now also J49.2 (Pin_2), J51.2 (Pin_2)
- no-connect marks 24 -> 28
Other:
- moved on the sheet: J48

Commit message: main2: ERC Check
Parts:
- J47, J48, J50: footprint Library:MAX_MX126-5.0-02P-GN01-Cu-S-A -> Connector_PinHeader_2.54mm:PinHeader_1x02_P2.54mm_Vertical
Changed lines of the file:
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@@
       (effects (font (size 1.27 1.27)) (justify left) hide)
     )
-    (property "Footprint" "Library:MAX_MX126-5.0-02P-GN01-Cu-S-A" (at 421.64 203.2 0)
+    (property "Footprint" "Connector_PinHeader_2.54mm:PinHeader_1x02_P2.54mm_Vertical" (at 421.64 203.2 0)
       (effects (font (size 1.27 1.27)) hide)
     )
@@
       (effects (font (size 1.27 1.27)) (justify left) hide)
     )
-    (property "Footprint" "Library:MAX_MX126-5.0-02P-GN01-Cu-S-A" (at 421.64 171.45 0)
+    (property "Footprint" "Connector_PinHeader_2.54mm:PinHeader_1x02_P2.54mm_Vertical" (at 421.64 171.45 0)
       (effects (font (size 1.27 1.27)) hide)
     )
@@
       (effects (font (size 1.27 1.27)) (justify left) hide)
     )
-    (property "Footprint" "Library:MAX_MX126-5.0-02P-GN01-Cu-S-A" (at 363.22 71.12 0)
+    (property "Footprint" "Connector_PinHeader_2.54mm:PinHeader_1x02_P2.54mm_Vertical" (at 363.22 71.12 0)
       (effects (font (size 1.27 1.27)) hide)
     )
