File: Cloud-Star-Lights-PCB/Cloud-Star-Lights-PCB.kicad_sch (KiCad schematic)
At the start: 175 parts, among them J1 Conn_01x02, J10 Conn_01x02, J11 Conn_01x02, J12 Conn_01x02, J13 Conn_01x02, J14 Conn_01x02, J15 Conn_01x02, J16 Conn_01x02, J17 Conn_01x02, J18 Conn_01x02, J19 Conn_01x02, J2 Conn_01x02, J20 Conn_01x02, J21 Conn_01x02, J22 Conn_01x02, J23 Conn_01x02, J24 Conn_01x02, J25 Conn_01x02, J26 Conn_01x02, J27 Conn_01x02, J28 Conn_01x02, J29 Conn_01x02, J3 Conn_01x02, J30 Conn_01x02, J31 Conn_01x04, J32 Conn_01x04, J33 Conn_01x04, J34 Conn_01x04, J35 Conn_01x04, J36 Conn_01x04, J37 Conn_01x04, J38 Conn_01x04, J39 Conn_01x04, J4 Conn_01x02, J40 Conn_01x04, J41 Conn_01x04, J42 Conn_01x04, J43 Conn_01x04, J44 Conn_01x04, J45 Conn_01x04, J46 Conn_01x02, J47 Conn_01x02, J48 Conn_01x02, J49 Screw_Terminal_01x02, J5 Conn_01x02, J50 Conn_01x02, J51 Screw_Terminal_01x02, J6 Conn_01x02, J7 Conn_01x02, J8 Conn_01x02, J9 Conn_01x02, Q1 2N3906, Q10 2N3906, Q11 2N3906, Q12 2N3906, Q13 2N3906, Q14 2N3906, Q15 2N3906, Q16 2N3906, Q17 2N3906, Q18 2N3906, Q19 2N3906, Q2 2N3906, Q20 2N3906, Q21 2N3906, Q22 2N3906, Q23 2N3906, Q24 2N3906, Q25 2N3906, Q26 2N3906, Q27 2N3906, Q28 2N3906, Q29 2N3906, Q3 2N3906, Q30 2N3906, Q31 2N3906, Q32 2N3906, Q33 2N3906, Q34 2N3906, Q35 2N3906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

Commit message: Schematic v2
Parts:
- removed J1, J10, J11, J12, J13, J14, J15, J16, J17, J18, J19, J2, J20, J21, J22, J23, J24, J25, J26, J27, J28, J29, J3, J30, J4, J5, J6, J7, J8, J9: Conn_01x02, Library:MAX_MX126-5.0-02P-GN01-Cu-S-A, symbol Connector_Generic:Conn_01x02
- removed J31, J32, J33, J34, J35, J36, J37, J38, J39, J40, J41, J42, J43, J44, J45: Conn_01x04, Library:JILN_JL301-50004U01, symbol Connector_Generic:Conn_01x04
- removed Q1, Q10, Q11, Q12, Q13, Q14, Q15, Q16, Q17, Q18, Q19, Q2, Q20, Q21, Q22, Q23, Q24, Q25, Q26, Q27, Q28, Q29, Q3, Q30, Q31, Q32, Q33, Q34, Q35, Q36, Q37, Q38, Q39, Q4, Q40, Q41, Q42, Q43, Q44, Q45, Q46, Q47, Q48, Q49, Q5, Q50, Q51, Q52, Q53, Q54, Q55, Q56, Q57, Q58, Q59, Q6, Q60, Q61, Q62, Q63, Q64, Q65, Q66, Q67, Q68, Q69, Q7, Q70, Q71, Q72, Q73, Q74, Q75, Q8, Q9: 2N3906, Package_TO_SOT_THT:TO-92S_Wide, symbol Transistor_BJT:2N3906
- removed R1, R10, R11, R12, R13, R14, R15, R16, R17, R18, R19, R2, R20, R21, R22, R23, R24, R25, R26, R27, R28, R29, R3, R30, R4, R5, R6, R7, R8, R9: 22Ω, Resistor_SMD:R_1206_3216Metric_Pad1.30x1.75mm_HandSolder, symbol Device:R
- removed R31, R34, R35: 10kΩ, Resistor_SMD:R_1206_3216Metric_Pad1.30x1.75mm_HandSolder, symbol Device:R
- removed U1, U3, U4: PCA9635, Package_SO:TSSOP-28_4.4x9.7mm_P0.65mm, symbol Driver_LED:PCA9635
- C1, C2, C4: value 10uf -> 0.1uF; footprint Capacitor_SMD:C_1206_3216Metric_Pad1.33x1.80mm_HandSolder -> Package_TO_SOT_THT:SOD-70_P5.08mm; now not fitted
- C3: now fitted
- R32, R33: value 10kΩ -> 3.3kΩ
Connections:
- net +3.3V: now also C2.1; no longer C1.2, C2.2, C4.2, U2.30 (VIN)
- net +5V: now also C4.1, U2.30 (VIN)
- net GND: now also C2.2, C4.2; no longer C2.1, C4.1
- net at C3.2, U2.16 (EN): now also C1.2
- net Control8: now reaches U2.15 (D23/VSPI_MOSI)
- net Control14: now reaches U2.19 (D34/ADC1_CH6)
- net Control15: now reaches U2.20 (D35/ADC1_CH7)
- net Control12: now reaches U2.21 (D32/ADC1_CH4/TOUCH9)
- net Control13: now reaches U2.22 (D33/ADC1_CH5/TOUCH8)
- net Control9: now reaches U2.23 (D25/ADC2_CH8/DAC1)
- net Control10: now reaches U2.24 (D26/ADC2_CH9/DAC2)
- net Control11: now reaches U2.25 (D27/ADC2_CH7/TOUCH7)
- net Control6: now reaches U2.26 (D14/ADC2_CH6/TOUCH6/HSPI_CLK)
- net Control4: now reaches U2.27 (D12/ADC2_CH5/TOUCH5/HSPI_MISO)
- net Control5: now reaches U2.28 (D13/ADC2_CH4/TOUCH4/HSPI_MOSI)
- net Control7: now reaches U2.3 (D15/ADC2_CH3/TOUCH3/HSPI_CS0)
- net Control1: now reaches U2.4 (D2/ADC2_CH2/TOUCH2)
- net Control2: now reaches U2.5 (D4/ADC2_CH0/TOUCH0)
- net Control3: now reaches U2.8 (D5/VSPI_CS0)
- no-connect marks 28 -> 10
Other:
- added sheet CloudController (CloudController.kicad_sch)
- added sheet CloudOutputs (CloudOutputs.kicad_sch)
- added sheet StarController1 (StarController1.kicad_sch)
- added sheet StarController2 (StarController1.kicad_sch)
- note added: "Cloud Notes: - 30 LEDs / 100cm - 20mA per 1 LED - 60mA / 10cm - Clouds have 90cm -> 540mA / 0.54A per channel Cloud Setup: - 15 clouds - Group clouds in groups of 3 - 5 cloud groups * 3 channels per group - 15 channels - Each channel should handle up to 2A TLDR: 15x 2A PWM channels"
- note added: "Microprocessor"
- note added: "Mounting Holes"
- note added: "Power"
- note added: "Star Notes: - IC has max 120ma per channel"
- note removed: "IC's"
- moved on the sheet: C5, C6, H1, H2, H3, H4, J46, J47, J48, J49, J50, J51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

Commit message: Update I2C addresses
Other:
- note added: "R: 1100 0001 = 0xC1 W: 1100 0000 = 0xC0"
- note added: "R: 1100 0011 = 0xC3 W: 1100 0010 = 0xC2"
Changed lines of the file:
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@@
+    (effects (font (size 1.27 1.27)) (justify left bottom))
+  )
+  (text "R: 1100 0001 = 0xC1\nW: 1100 0000 = 0xC0" (at 41.91 92.71 0)
     (effects (font (size 1.27 1.27)) (justify left bottom))
   )
@@
     (effects (font (size 6 6)) (justify left bottom))
   )
+  (text "R: 1100 0011 = 0xC3\nW: 1100 0010 = 0xC2" (at 80.01 92.71 0)
+    (effects (font (size 1.27 1.27)) (justify left bottom))
+  )
   (label "Control4" (at 43.18 205.74 0) (fields_autoplaced)

Commit message: Routing
Connections:
- net Control14: now also U2.9 (D18/VSPI_CLK); no longer U2.19 (D34/ADC1_CH6)
- net Control15: now also U2.10 (D19/VSPI_MISO); no longer U2.20 (D35/ADC1_CH7)
- net Control3: now also U2.7 (TX2/D17); no longer U2.8 (D5/VSPI_CS0)
Other:
- moved on the sheet: J46, R32, R33

Commit message: Finalize rev2 order
- added comments, silk screens
- exported PDF and gerber
Other:
- note added: "TODO: these control labels should have the color included in them"
Changed lines of the file:
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@@
     (effects (font (size 6 6)) (justify left bottom))
+  )
+  (text "TODO: these control labels should\nhave the color included in them"
+    (at 203.2 100.33 0)
+    (effects (font (size 1.27 1.27)) (justify left bottom))
   )
   (text "Star Notes:\n - IC has max 120ma per channel" (at 34.29 46.99 0)
