File: Cloud-Star-Lights-PCB/Cloud-Star-Lights-PCB.kicad_pcb (KiCad board)
At the start: 2 copper layers, 78 parts, among them U2 PCA9685PW, U3 PCA9685PW

Commit message: Comments
Parts:
- added Q31: 2N3906, Package_TO_SOT_THT:TO-92_Inline, F.Cu at (119.6, 45.2)
- added Q32: 2N3906, Package_TO_SOT_THT:TO-92_Inline, F.Cu at (119.6, 50.9)
- added Q33: 2N3906, Package_TO_SOT_THT:TO-92_Inline, F.Cu at (119.6, 56.7)
- added Q34: 2N3906, Package_TO_SOT_THT:TO-92_Inline, F.Cu at (126.1, 33.6)
- added Q35: 2N3906, Package_TO_SOT_THT:TO-92_Inline, F.Cu at (126.1, 39.4)
- added Q36: 2N3906, Package_TO_SOT_THT:TO-92_Inline, F.Cu at (126.1, 45.2)
- added Q37: ~, Library:AP5N10S, F.Cu at (82.8, 87.6)
- added Q38: ~, Library:AP5N10S, F.Cu at (82.8, 91.1)
- added Q39: ~, Library:AP5N10S, F.Cu at (82.8, 94.7)
- added Q40: ~, Library:AP5N10S, F.Cu at (82.8, 98.2)
- added Q41: ~, Library:AP5N10S, F.Cu at (82.8, 101.8)
- added Q42: ~, Library:AP5N10S, F.Cu at (82.8, 105.3)
- added Q43: ~, Library:AP5N10S, F.Cu at (82.8, 108.9)
- added Q44: ~, Library:AP5N10S, F.Cu at (82.8, 112.4)
- added Q45: ~, Library:AP5N10S, F.Cu at (82.8, 116.0)
- added Q46: 2N3906, Package_TO_SOT_THT:TO-92_Inline, F.Cu at (126.1, 50.9)
- added Q47: 2N3906, Package_TO_SOT_THT:TO-92_Inline, F.Cu at (126.1, 56.7)
- added Q48: 2N3906, Package_TO_SOT_THT:TO-92_Inline, F.Cu at (132.6, 33.6)
- added Q49: 2N3906, Package_TO_SOT_THT:TO-92_Inline, F.Cu at (132.6, 39.4)
- added Q50: 2N3906, Package_TO_SOT_THT:TO-92_Inline, F.Cu at (132.6, 45.2)
- added Q51: 2N3906, Package_TO_SOT_THT:TO-92_Inline, F.Cu at (132.6, 50.9)
- added Q52: ~, Library:AP5N10S, F.Cu at (86.7, 87.6)
- added Q53: ~, Library:AP5N10S, F.Cu at (86.7, 91.1)
- added Q54: ~, Library:AP5N10S, F.Cu at (86.7, 94.7)
- added Q55: ~, Library:AP5N10S, F.Cu at (86.7, 98.2)
- added Q56: ~, Library:AP5N10S, F.Cu at (86.7, 101.8)
- added Q57: ~, Library:AP5N10S, F.Cu at (86.7, 105.3)
- added Q58: ~, Library:AP5N10S, F.Cu at (86.7, 108.9)
- added Q59: ~, Library:AP5N10S, F.Cu at (86.7, 112.4)
- added Q60: ~, Library:AP5N10S, F.Cu at (86.7, 116.0)
- added Q61: 2N3906, Package_TO_SOT_THT:TO-92_Inline, F.Cu at (132.6, 56.7)
- added Q62: 2N3906, Package_TO_SOT_THT:TO-92_Inline, F.Cu at (139.1, 33.6)
- added Q63: 2N3906, Package_TO_SOT_THT:TO-92_Inline, F.Cu at (139.1, 39.4)
- added Q64: 2N3906, Package_TO_SOT_THT:TO-92_Inline, F.Cu at (139.1, 45.2)
- added Q65: 2N3906, Package_TO_SOT_THT:TO-92_Inline, F.Cu at (139.1, 50.9)
- added Q66: 2N3906, Package_TO_SOT_THT:TO-92_Inline, F.Cu at (139.1, 56.7)
- added Q67: ~, Library:AP5N10S, F.Cu at (90.6, 87.6)
- added Q68: ~, Library:AP5N10S, F.Cu at (90.6, 91.1)
- added Q69: ~, Library:AP5N10S, F.Cu at (90.6, 94.7)
- added Q70: ~, Library:AP5N10S, F.Cu at (90.6, 98.2)
- added Q71: ~, Library:AP5N10S, F.Cu at (90.6, 101.8)
- added Q72: ~, Library:AP5N10S, F.Cu at (90.6, 105.3)
- added Q73: ~, Library:AP5N10S, F.Cu at (90.6, 108.9)
- added Q74: ~, Library:AP5N10S, F.Cu at (90.6, 112.4)
- added Q75: ~, Library:AP5N10S, F.Cu at (90.6, 116.0)
- added R1: ~, Resistor_SMD:R_0201_0603Metric_Pad0.64x0.40mm_HandSolder, F.Cu at (155.4, 27.9)
- added R10: ~, Resistor_SMD:R_0201_0603Metric_Pad0.64x0.40mm_HandSolder, F.Cu at (108.8, 110.4)
- added R11: ~, Resistor_SMD:R_0201_0603Metric_Pad0.64x0.40mm_HandSolder, F.Cu at (108.8, 112.1)
- added R12: ~, Resistor_SMD:R_0201_0603Metric_Pad0.64x0.40mm_HandSolder, F.Cu at (108.8, 113.9)
- added R13: ~, Resistor_SMD:R_0201_0603Metric_Pad0.64x0.40mm_HandSolder, F.Cu at (111.6, 105.1)
- added R14: ~, Resistor_SMD:R_0201_0603Metric_Pad0.64x0.40mm_HandSolder, F.Cu at (111.6, 106.9)
- added R15: ~, Resistor_SMD:R_0201_0603Metric_Pad0.64x0.40mm_HandSolder, F.Cu at (111.6, 108.6)
- added R16: ~, Resistor_SMD:R_0201_0603Metric_Pad0.64x0.40mm_HandSolder, F.Cu at (111.6, 110.4)
- added R17: ~, Resistor_SMD:R_0201_0603Metric_Pad0.64x0.40mm_HandSolder, F.Cu at (111.6, 112.1)
- added R18: ~, Resistor_SMD:R_0201_0603Metric_Pad0.64x0.40mm_HandSolder, F.Cu at (111.6, 113.9)
- added R19: ~, Resistor_SMD:R_0201_0603Metric_Pad0.64x0.40mm_HandSolder, F.Cu at (114.4, 105.1)
- added R2: ~, Resistor_SMD:R_0201_0603Metric_Pad0.64x0.40mm_HandSolder, F.Cu at (106.0, 106.9)
- added R20: ~, Resistor_SMD:R_0201_0603Metric_Pad0.64x0.40mm_HandSolder, F.Cu at (114.4, 106.9)
- added R21: ~, Resistor_SMD:R_0201_0603Metric_Pad0.64x0.40mm_HandSolder, F.Cu at (114.4, 108.6)
- added R22: ~, Resistor_SMD:R_0201_0603Metric_Pad0.64x0.40mm_HandSolder, F.Cu at (114.4, 110.4)
- added R23: ~, Resistor_SMD:R_0201_0603Metric_Pad0.64x0.40mm_HandSolder, F.Cu at (114.4, 112.1)
- added R24: ~, Resistor_SMD:R_0201_0603Metric_Pad0.64x0.40mm_HandSolder, F.Cu at (114.4, 113.9)
- added R25: ~, Resistor_SMD:R_0201_0603Metric_Pad0.64x0.40mm_HandSolder, F.Cu at (117.2, 105.1)
- added R26: ~, Resistor_SMD:R_0201_0603Metric_Pad0.64x0.40mm_HandSolder, F.Cu at (117.2, 106.9)
- added R27: ~, Resistor_SMD:R_0201_0603Metric_Pad0.64x0.40mm_HandSolder, F.Cu at (117.2, 108.6)
- added R28: ~, Resistor_SMD:R_0201_0603Metric_Pad0.64x0.40mm_HandSolder, F.Cu at (117.2, 110.4)
- added R29: ~, Resistor_SMD:R_0201_0603Metric_Pad0.64x0.40mm_HandSolder, F.Cu at (117.2, 112.1)
- added R3: ~, Resistor_SMD:R_0201_0603Metric_Pad0.64x0.40mm_HandSolder, F.Cu at (106.0, 108.6)
- added R30: ~, Resistor_SMD:R_0201_0603Metric_Pad0.64x0.40mm_HandSolder, F.Cu at (117.2, 113.9)
- added R4: ~, Resistor_SMD:R_0201_0603Metric_Pad0.64x0.40mm_HandSolder, F.Cu at (106.0, 110.4)
- added R5: ~, Resistor_SMD:R_0201_0603Metric_Pad0.64x0.40mm_HandSolder, F.Cu at (106.0, 112.1)
- added R6: ~, Resistor_SMD:R_0201_0603Metric_Pad0.64x0.40mm_HandSolder, F.Cu at (106.0, 113.9)
- added R7: ~, Resistor_SMD:R_0201_0603Metric_Pad0.64x0.40mm_HandSolder, F.Cu at (108.8, 105.1)
- added R8: ~, Resistor_SMD:R_0201_0603Metric_Pad0.64x0.40mm_HandSolder, F.Cu at (108.8, 106.9)
- added R9: ~, Resistor_SMD:R_0201_0603Metric_Pad0.64x0.40mm_HandSolder, F.Cu at (108.8, 108.6)
- added U1: ESP32-Module-30Pin, Library:ESP32-Module-30Pin, F.Cu at (50.8, 58.4)
- added U4: PCA9685PW, Package_SO:TSSOP-28_4.4x9.7mm_P0.65mm, F.Cu at (144.5, 110.1)
- J1: footprint Library:0353120460 -> Library:Cixi_Kefa_Elec_KF135T-10.16-3P
- J10, J17, J18, J19, J26, J27, J28, J35, J36, J37, J44, J45, J8, J9: footprint Library:0353120460 -> Library:JILN_JL301-50004U01
- J11, J12, J13, J14, J15, J16, J2, J20, J21, J22, J23, J24, J25, J29, J3, J30, J31, J32, J33, J34, J38, J39, J4, J40, J41, J42, J43, J5, J6, J7: footprint Library:0353120460 -> Library:MAX_MX126-5.0-02P-GN01-Cu-S-A
- J46: footprint Library:Cixi_Kefa_Elec_KF135T-10.16-3P -> Library:JILN_JL301-50004U01
- Q10, Q11, Q12, Q13, Q14, Q15, Q25, Q26, Q27, Q28, Q29, Q30: value ~ -> 2N3906; footprint Library:AP5N10S -> Package_TO_SOT_THT:TO-92_Inline
- moved U3 99.0 mm to (135.7, 110.1)
- moved Q21 93.6 mm to (78.9, 105.3)
- moved Q22 93.6 mm to (78.9, 108.9)
- moved Q23 93.6 mm to (78.9, 112.4)
- moved Q24 93.6 mm to (78.9, 116.0)
- moved U2 92.2 mm to (127.0, 110.1)
- moved Q6 87.1 mm to (75.0, 105.3)
- moved Q7 87.1 mm to (75.0, 108.9)
- moved Q8 87.1 mm to (75.0, 112.4)
- moved Q9 87.1 mm to (75.0, 116.0)
- moved Q16 81.8 mm to (78.9, 87.6)
- moved Q17 81.8 mm to (78.9, 91.1)
- moved Q18 81.8 mm to (78.9, 94.7)
- moved Q19 81.8 mm to (78.9, 98.2)
- moved Q20 81.8 mm to (78.9, 101.8)
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Connections:
- J1 pad 1: +5V -> +3.3V
- J1 pad 2: /Clouds_Power_R1 -> +5V
- J1 pad 3: /Clouds_Power_G1 -> GNDREF
- J10 pad 1: +5V -> Net-(Q7-C)
- J10 pad 2: /Clouds_Power_R5 -> Net-(Q8-C)
- J10 pad 3: /Clouds_Power_G5 -> Net-(Q9-C)
- J10 pad 4: /Clouds_Power_B5 -> +5V
- J11 pad 1: +5V -> Net-(J11-Pad1)
- J11 pad 2: /Clouds_Power_R2 -> GNDREF
- J12 pad 1: +5V -> Net-(J12-Pad1)
- J12 pad 2: /Clouds_Power_R3 -> GNDREF
- J13 pad 1: +5V -> Net-(J13-Pad1)
- J13 pad 2: /Clouds_Power_R5 -> GNDREF
- J14 pad 1: +5V -> Net-(J14-Pad1)
- J14 pad 2: /Clouds_Power_R4 -> GNDREF
- J15 pad 1: +5V -> Net-(J15-Pad1)
- J15 pad 2: /Clouds_Power_R5 -> GNDREF
- J16 pad 1: +5V -> Net-(J16-Pad1)
- J16 pad 2: /Stars_Power_R1 -> GNDREF
- J17 pad 1: +5V -> Net-(Q16-C)
- J17 pad 2: /Stars_Power_R2 -> Net-(Q17-C)
- J17 pad 3: /Stars_Power_G2 -> Net-(Q18-C)
- J17 pad 4: /Stars_Power_B2 -> +5V
- J18 pad 1: +5V -> Net-(Q19-C)
- J18 pad 2: /Stars_Power_R3 -> Net-(Q20-C)
- J18 pad 3: /Stars_Power_G3 -> Net-(Q21-C)
- J18 pad 4: /Stars_Power_B3 -> +5V
- J19 pad 1: +5V -> Net-(Q22-C)
- J19 pad 2: /Stars_Power_R4 -> Net-(Q23-C)
- J19 pad 3: /Stars_Power_G4 -> Net-(Q24-C)
- J19 pad 4: /Stars_Power_B4 -> +5V
- J2 pad 1: +5V -> Net-(J2-Pad1)
- J2 pad 2: /Clouds_Power_R1 -> GNDREF
- J20 pad 1: +5V -> Net-(J20-Pad1)
- J20 pad 2: /Stars_Power_R5 -> GNDREF
- J21 pad 1: +5V -> Net-(J21-Pad1)
- J21 pad 2: /Stars_Power_R1 -> GNDREF
- J22 pad 1: +5V -> Net-(J22-Pad1)
- J22 pad 2: /Stars_Power_R2 -> GNDREF
- J23 pad 1: +5V -> Net-(J23-Pad1)
- J23 pad 2: /Stars_Power_R3 -> GNDREF
- J24 pad 1: +5V -> Net-(J24-Pad1)
- J24 pad 2: /Stars_Power_R4 -> GNDREF
- J25 pad 1: +5V -> Net-(J25-Pad1)
- J25 pad 2: /Stars_Power_R5 -> GNDREF
- J26 pad 1: +5V -> Net-(Q37-C)
- J26 pad 2: /Stars_Power_R1 -> Net-(Q38-C)
- J26 pad 3: /Stars_Power_G1 -> Net-(Q39-C)
- J26 pad 4: /Stars_Power_B1 -> +5V
- J27 pad 1: +5V -> Net-(Q40-C)
- J27 pad 2: /Stars_Power_R2 -> Net-(Q41-C)
- J27 pad 3: /Stars_Power_G2 -> Net-(Q42-C)
- J27 pad 4: /Stars_Power_B2 -> +5V
- J28 pad 1: +5V -> Net-(Q43-C)
- J28 pad 2: /Stars_Power_R3 -> Net-(Q44-C)
- J28 pad 3: /Stars_Power_G3 -> Net-(Q45-C)
- J28 pad 4: /Stars_Power_B3 -> +5V
- J29 pad 1: +5V -> Net-(J29-Pad1)
- J29 pad 2: /Stars_Power_R4 -> GNDREF
- J3 pad 1: +5V -> Net-(J3-Pad1)
- J3 pad 2: /Clouds_Power_R1 -> GNDREF
- J30 pad 1: +5V -> Net-(J30-Pad1)
- J30 pad 2: /Stars_Power_R5 -> GNDREF
- J31 pad 1: +5V -> Net-(J31-Pad1)
- J31 pad 2: /Stars_Power_R1 -> GNDREF
- J32 pad 1: +5V -> Net-(J32-Pad1)
- J32 pad 2: /Stars_Power_R2 -> GNDREF
- J33 pad 1: +5V -> Net-(J33-Pad1)
- J33 pad 2: /Stars_Power_R3 -> GNDREF
- J34 pad 1: +5V -> Net-(J34-Pad1)
- J34 pad 2: /Stars_Power_R4 -> GNDREF
- J35 pad 1: +5V -> Net-(Q52-C)
- J35 pad 2: /Stars_Power_R5 -> Net-(Q53-C)
- J35 pad 3: /Stars_Power_G5 -> Net-(Q54-C)
- J35 pad 4: /Stars_Power_B5 -> +5V
- J36 pad 1: +5V -> Net-(Q55-C)
- J36 pad 2: /Stars_Power_R1 -> Net-(Q56-C)
- J36 pad 3: /Stars_Power_G1 -> Net-(Q57-C)
- J36 pad 4: /Stars_Power_B1 -> +5V
- J37 pad 1: +5V -> Net-(Q58-C)
- J37 pad 2: /Stars_Power_R2 -> Net-(Q59-C)
- J37 pad 3: /Stars_Power_G2 -> Net-(Q60-C)
- J37 pad 4: /Stars_Power_B2 -> +5V
- J38 pad 1: +5V -> Net-(J38-Pad1)
- J38 pad 2: /Stars_Power_R3 -> GNDREF
- J39 pad 1: +5V -> Net-(J39-Pad1)
- J39 pad 2: /Stars_Power_R4 -> GNDREF
- J4 pad 1: +5V -> Net-(J4-Pad1)
- J4 pad 2: /Clouds_Power_R2 -> GNDREF
- J40 pad 1: +5V -> Net-(J40-Pad1)
- J40 pad 2: /Stars_Power_R5 -> GNDREF
- J41 pad 1: +5V -> Net-(J41-Pad1)
- J41 pad 2: /Stars_Power_R1 -> GNDREF
- J42 pad 1: +5V -> Net-(J42-Pad1)
- J42 pad 2: /Stars_Power_R2 -> GNDREF
- J43 pad 1: +5V -> Net-(J43-Pad1)
- J43 pad 2: /Stars_Power_R3 -> GNDREF
- J44 pad 1: +5V -> Net-(Q67-C)
- J44 pad 2: /Stars_Power_R4 -> Net-(Q68-C)
- J44 pad 3: /Stars_Power_G4 -> Net-(Q69-C)
- J44 pad 4: /Stars_Power_B4 -> +5V
- J45 pad 1: +5V -> Net-(Q70-C)
- J45 pad 2: /Stars_Power_R5 -> Net-(Q71-C)
- J45 pad 3: /Stars_Power_G5 -> Net-(Q72-C)
- J45 pad 4: /Stars_Power_B5 -> +5V
- J46 pad 1: +3.3V -> Net-(Q73-C)
- J46 pad 2: +5V -> Net-(Q74-C)
- J46 pad 3: GNDREF -> Net-(Q75-C)
- J5 pad 1: +5V -> Net-(J5-Pad1)
- J5 pad 2: /Clouds_Power_R2 -> GNDREF
- J6 pad 1: +5V -> Net-(J6-Pad1)
- J6 pad 2: /Clouds_Power_R3 -> GNDREF
- J7 pad 1: +5V -> Net-(J7-Pad1)
- J7 pad 2: /Clouds_Power_R3 -> GNDREF
- J8 pad 1: +5V -> Net-(Q1-C)
- J8 pad 2: /Clouds_Power_R4 -> Net-(Q2-C)
- J8 pad 3: /Clouds_Power_G4 -> Net-(Q3-C)
- J8 pad 4: /Clouds_Power_B4 -> +5V
- J9 pad 1: +5V -> Net-(Q4-C)
- J9 pad 2: /Clouds_Power_R4 -> Net-(Q5-C)
- J9 pad 3: /Clouds_Power_G4 -> Net-(Q6-C)
- J9 pad 4: /Clouds_Power_B4 -> +5V
- Q1 pad 1: /Clouds_Control_R1 -> /Cloud_Control_R1
- Q1 pad 2: (no net) -> Net-(Q1-C)
- Q1 pad 3: (no net) -> GNDREF
- Q10 pad 1: /Clouds_Control_G5 -> +5V
- Q10 pad 2: (no net) -> /Star_Control_1
- Q10 pad 3: (no net) -> Net-(Q10-C)
- Q11 pad 1: /Clouds_Control_B1 -> +5V
- Q11 pad 2: (no net) -> /Star_Control_6
- Q11 pad 3: (no net) -> Net-(Q11-C)
- Q12 pad 1: /Clouds_Control_B2 -> +5V
- Q12 pad 2: (no net) -> /Star_Control_11
- Q12 pad 3: (no net) -> Net-(Q12-C)
- Q13 pad 1: /Clouds_Control_B3 -> +5V
- Q13 pad 2: (no net) -> /Star_Control_16
- Q13 pad 3: (no net) -> Net-(Q13-C)
- Q14 pad 1: /Clouds_Control_B4 -> +5V
- Q14 pad 2: (no net) -> /Star_Control_21
- Q14 pad 3: (no net) -> Net-(Q14-C)
- Q15 pad 1: /Clouds_Control_B5 -> +5V
- Q15 pad 2: (no net) -> /Star_Control_26
- Q15 pad 3: (no net) -> Net-(Q15-C)
- Q16 pad 1: /Stars_Control_R1 -> /Cloud_Control_R2
- Q16 pad 2: (no net) -> Net-(Q16-C)
- Q16 pad 3: (no net) -> GNDREF
- Q17 pad 1: /Stars_Control_R2 -> /Cloud_Control_G2
- Q17 pad 2: (no net) -> Net-(Q17-C)
- Q17 pad 3: (no net) -> GNDREF
- Q18 pad 1: /Stars_Control_R3 -> /Cloud_Control_B2
- Q18 pad 2: (no net) -> Net-(Q18-C)
- Q18 pad 3: (no net) -> GNDREF
- Q19 pad 1: /Stars_Control_R4 -> /Cloud_Control_R2
- Q19 pad 2: (no net) -> Net-(Q19-C)
- Q19 pad 3: (no net) -> GNDREF
- Q2 pad 1: /Clouds_Control_R2 -> /Cloud_Control_G1
- Q2 pad 2: (no net) -> Net-(Q2-C)
- Q2 pad 3: (no net) -> GNDREF
- Q20 pad 1: /Stars_Control_R5 -> /Cloud_Control_G2
- Q20 pad 2: (no net) -> Net-(Q20-C)
- Q20 pad 3: (no net) -> GNDREF
- Q21 pad 1: /Stars_Control_G1 -> /Cloud_Control_B2
- Q21 pad 2: (no net) -> Net-(Q21-C)
- Q21 pad 3: (no net) -> GNDREF
- Q22 pad 1: /Stars_Control_G2 -> /Cloud_Control_R2
- Q22 pad 2: (no net) -> Net-(Q22-C)
- Q22 pad 3: (no net) -> GNDREF
- Q23 pad 1: /Stars_Control_G3 -> /Cloud_Control_G2
- Q23 pad 2: (no net) -> Net-(Q23-C)
- Q23 pad 3: (no net) -> GNDREF
- Q24 pad 1: /Stars_Control_G4 -> /Cloud_Control_B2
- Q24 pad 2: (no net) -> Net-(Q24-C)
- Q24 pad 3: (no net) -> GNDREF
- Q25 pad 1: /Stars_Control_G5 -> +5V
- Q25 pad 2: (no net) -> /Star_Control_2
- Q25 pad 3: (no net) -> Net-(Q25-C)
- Q26 pad 1: /Stars_Control_B1 -> +5V
- Q26 pad 2: (no net) -> /Star_Control_7
- Q26 pad 3: (no net) -> Net-(Q26-C)
- Q27 pad 1: /Stars_Control_B2 -> +5V
- Q27 pad 2: (no net) -> /Star_Control_12
- Q27 pad 3: (no net) -> Net-(Q27-C)
- Q28 pad 1: /Stars_Control_B3 -> +5V
- Q28 pad 2: (no net) -> /Star_Control_17
- Q28 pad 3: (no net) -> Net-(Q28-C)
- Q29 pad 1: /Stars_Control_B4 -> +5V
- Q29 pad 2: (no net) -> /Star_Control_22
- Q29 pad 3: (no net) -> Net-(Q29-C)
- Q3 pad 1: /Clouds_Control_R3 -> /Cloud_Control_B1
- Q3 pad 2: (no net) -> Net-(Q3-C)
- Q3 pad 3: (no net) -> GNDREF
- Q30 pad 1: /Stars_Control_B5 -> +5V
- Q30 pad 2: (no net) -> /Star_Control_27
- Q30 pad 3: (no net) -> Net-(Q30-C)
- Q4 pad 1: /Clouds_Control_R4 -> /Cloud_Control_R1
- Q4 pad 2: (no net) -> Net-(Q4-C)
- Q4 pad 3: (no net) -> GNDREF
- Q5 pad 1: /Clouds_Control_R5 -> /Cloud_Control_G1
- Q5 pad 2: (no net) -> Net-(Q5-C)
- Q5 pad 3: (no net) -> GNDREF
- Q6 pad 1: /Clouds_Control_G1 -> /Cloud_Control_B1
- Q6 pad 2: (no net) -> Net-(Q6-C)
- Q6 pad 3: (no net) -> GNDREF
- Q7 pad 1: /Clouds_Control_G2 -> /Cloud_Control_R1
- Q7 pad 2: (no net) -> Net-(Q7-C)
- Q7 pad 3: (no net) -> GNDREF
- Q8 pad 1: /Clouds_Control_G3 -> /Cloud_Control_G1
- Q8 pad 2: (no net) -> Net-(Q8-C)
- Q8 pad 3: (no net) -> GNDREF
- Q9 pad 1: /Clouds_Control_G4 -> /Cloud_Control_B1
- Q9 pad 2: (no net) -> Net-(Q9-C)
- Q9 pad 3: (no net) -> GNDREF
- U2 pad 10: /Clouds_Control_G2 -> /Star_Control_5
- U2 pad 11: /Clouds_Control_B2 -> /Star_Control_6
- U2 pad 12: /Clouds_Control_R3 -> /Star_Control_7
- U2 pad 13: /Clouds_Control_G3 -> /Star_Control_8
- U2 pad 15: /Clouds_Control_B3 -> /Star_Control_9
- U2 pad 16: /Clouds_Control_R4 -> /Star_Control_10
- U2 pad 17: /Clouds_Control_G4 -> /Star_Control_11
- U2 pad 18: /Clouds_Control_B4 -> /Star_Control_12
- U2 pad 19: /Clouds_Control_R5 -> /Star_Control_13
- U2 pad 20: /Clouds_Control_G5 -> /Star_Control_14
- U2 pad 21: /Clouds_Control_B5 -> /Star_Control_15
- U2 pad 6: /Clouds_Control_R1 -> /Star_Control_1
- U2 pad 7: /Clouds_Control_G1 -> /Star_Control_2
- U2 pad 8: /Clouds_Control_B1 -> /Star_Control_3
- U2 pad 9: /Clouds_Control_R2 -> /Star_Control_4
- U3 pad 10: /Stars_Control_G2 -> /Star_Control_20
- U3 pad 11: /Stars_Control_B2 -> /Star_Control_21
- U3 pad 12: /Stars_Control_R3 -> /Star_Control_22
- U3 pad 13: /Stars_Control_G3 -> /Star_Control_23
- U3 pad 15: /Stars_Control_B3 -> /Star_Control_24
- U3 pad 16: /Stars_Control_R4 -> /Star_Control_25
- U3 pad 17: /Stars_Control_G4 -> /Star_Control_26
- U3 pad 18: /Stars_Control_B4 -> /Star_Control_27
- U3 pad 19: /Stars_Control_R5 -> /Star_Control_28
- U3 pad 20: /Stars_Control_G5 -> /Star_Control_29
- U3 pad 21: /Stars_Control_B5 -> /Star_Control_30
- U3 pad 5: +3.3V -> GNDREF
- U3 pad 6: /Stars_Control_R1 -> /Star_Control_16
- U3 pad 7: /Stars_Control_G1 -> /Star_Control_17
- U3 pad 8: /Stars_Control_B1 -> /Star_Control_18
- U3 pad 9: /Stars_Control_R2 -> /Star_Control_19

Commit message: Schematic
Parts:
- added C1: 10uf, Capacitor_SMD:C_0201_0603Metric_Pad0.64x0.40mm_HandSolder, F.Cu at (172.4, 122.7)
- added C2: 10uf, Capacitor_SMD:C_0201_0603Metric_Pad0.64x0.40mm_HandSolder, F.Cu at (172.4, 124.5)
- added C3: 0.1uF, Capacitor_SMD:C_0201_0603Metric_Pad0.64x0.40mm_HandSolder, F.Cu at (172.4, 126.2)
- added C4: 10uf, Capacitor_SMD:C_0201_0603Metric_Pad0.64x0.40mm_HandSolder, F.Cu at (172.4, 128.0)
- added C5: 0.1uF, Capacitor_SMD:C_0201_0603Metric_Pad0.64x0.40mm_HandSolder, F.Cu at (172.4, 129.7)
- added C6: 0.1uF, Capacitor_SMD:C_0201_0603Metric_Pad0.64x0.40mm_HandSolder, F.Cu at (172.4, 131.5)
- added J47: Conn_01x02, Library:MAX_MX126-5.0-02P-GN01-Cu-S-A, F.Cu at (147.4, 121.0)
- added J48: Conn_01x02, Library:MAX_MX126-5.0-02P-GN01-Cu-S-A, F.Cu at (147.4, 124.0)
- added J49: Conn_01x03, Library:Cixi_Kefa_Elec_KF135T-10.16-3P, F.Cu at (73.7, 160.0)
- added J50: Conn_01x02, Library:MAX_MX126-5.0-02P-GN01-Cu-S-A, F.Cu at (147.4, 127.0)
- added R31: 10kΩ, Resistor_SMD:R_0201_0603Metric_Pad0.64x0.40mm_HandSolder, F.Cu at (186.5, 124.5)
- added R32: 10kΩ, Resistor_SMD:R_0201_0603Metric_Pad0.64x0.40mm_HandSolder, F.Cu at (186.5, 126.2)
- added R33: 10kΩ, Resistor_SMD:R_0201_0603Metric_Pad0.64x0.40mm_HandSolder, F.Cu at (186.5, 128.0)
- added R34: 10kΩ, Resistor_SMD:R_0201_0603Metric_Pad0.64x0.40mm_HandSolder, F.Cu at (186.5, 129.7)
- added R35: 10kΩ, Resistor_SMD:R_0201_0603Metric_Pad0.64x0.40mm_HandSolder, F.Cu at (186.5, 131.5)
- J1: value ~ -> Conn_01x02; footprint Library:Cixi_Kefa_Elec_KF135T-10.16-3P -> Library:MAX_MX126-5.0-02P-GN01-Cu-S-A
- J10, J17, J18, J19, J26, J27, J28, J46, J8, J9: value ~ -> Conn_01x02; footprint Library:JILN_JL301-50004U01 -> Library:MAX_MX126-5.0-02P-GN01-Cu-S-A
- J11, J12, J13, J14, J15, J16, J2, J20, J21, J22, J23, J24, J25, J29, J3, J30, J4, J5, J6, J7: value ~ -> Conn_01x02
- J31, J32, J33, J34, J38, J39, J40, J41, J42, J43: value ~ -> Conn_01x04; footprint Library:MAX_MX126-5.0-02P-GN01-Cu-S-A -> Library:JILN_JL301-50004U01
- J35, J36, J37, J44, J45: value ~ -> Conn_01x04
- Q1, Q16, Q17, Q18, Q19, Q2, Q20, Q21, Q22, Q23, Q24, Q3, Q37, Q38, Q39, Q4, Q40, Q41, Q42, Q43, Q44, Q45, Q5, Q52, Q53, Q54, Q55, Q56, Q57, Q58, Q59, Q6, Q60, Q67, Q68, Q69, Q7, Q70, Q71, Q72, Q73, Q74, Q75, Q8, Q9: value ~ -> 2N3906; footprint Library:AP5N10S -> Package_TO_SOT_THT:TO-92_Inline
- R1, R10, R11, R12, R13, R14, R15, R16, R17, R18, R19, R2, R20, R21, R22, R23, R24, R25, R26, R27, R28, R29, R3, R30, R4, R5, R6, R7, R8, R9: value ~ -> 22Ω
- U1: value ESP32-Module-30Pin -> PCA9635; footprint Library:ESP32-Module-30Pin -> Package_SO:TSSOP-28_4.4x9.7mm_P0.65mm
- U2: value PCA9685PW -> ESP32-Module-30Pin; footprint Package_SO:TSSOP-28_4.4x9.7mm_P0.65mm -> Library:ESP32-Module-30Pin
- U3, U4: value PCA9685PW -> PCA9635
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Connections:
- J1 pad 1: +3.3V -> Net-(J1-Pin_1)
- J1 pad 2: +5V -> Net-(J1-Pin_2)
- J10 pad 1: Net-(Q7-C) -> Net-(J10-Pin_1)
- J10 pad 2: Net-(Q8-C) -> Net-(J10-Pin_2)
- J11 pad 1: Net-(J11-Pad1) -> Net-(J11-Pin_1)
- J11 pad 2: GNDREF -> Net-(J11-Pin_2)
- J12 pad 1: Net-(J12-Pad1) -> Net-(J12-Pin_1)
- J12 pad 2: GNDREF -> Net-(J12-Pin_2)
- J13 pad 1: Net-(J13-Pad1) -> Net-(J13-Pin_1)
- J13 pad 2: GNDREF -> Net-(J13-Pin_2)
- J14 pad 1: Net-(J14-Pad1) -> Net-(J14-Pin_1)
- J14 pad 2: GNDREF -> Net-(J14-Pin_2)
- J15 pad 1: Net-(J15-Pad1) -> Net-(J15-Pin_1)
- J15 pad 2: GNDREF -> Net-(J15-Pin_2)
- J16 pad 1: Net-(J16-Pad1) -> Net-(J16-Pin_1)
- J16 pad 2: GNDREF -> Net-(J16-Pin_2)
- J17 pad 1: Net-(Q16-C) -> Net-(J17-Pin_1)
- J17 pad 2: Net-(Q17-C) -> Net-(J17-Pin_2)
- J18 pad 1: Net-(Q19-C) -> Net-(J18-Pin_1)
- J18 pad 2: Net-(Q20-C) -> Net-(J18-Pin_2)
- J19 pad 1: Net-(Q22-C) -> Net-(J19-Pin_1)
- J19 pad 2: Net-(Q23-C) -> Net-(J19-Pin_2)
- J2 pad 1: Net-(J2-Pad1) -> Net-(J2-Pin_1)
- J2 pad 2: GNDREF -> Net-(J2-Pin_2)
- J20 pad 1: Net-(J20-Pad1) -> Net-(J20-Pin_1)
- J20 pad 2: GNDREF -> Net-(J20-Pin_2)
- J21 pad 1: Net-(J21-Pad1) -> Net-(J21-Pin_1)
- J21 pad 2: GNDREF -> Net-(J21-Pin_2)
- J22 pad 1: Net-(J22-Pad1) -> Net-(J22-Pin_1)
- J22 pad 2: GNDREF -> Net-(J22-Pin_2)
- J23 pad 1: Net-(J23-Pad1) -> Net-(J23-Pin_1)
- J23 pad 2: GNDREF -> Net-(J23-Pin_2)
- J24 pad 1: Net-(J24-Pad1) -> Net-(J24-Pin_1)
- J24 pad 2: GNDREF -> Net-(J24-Pin_2)
- J25 pad 1: Net-(J25-Pad1) -> Net-(J25-Pin_1)
- J25 pad 2: GNDREF -> Net-(J25-Pin_2)
- J26 pad 1: Net-(Q37-C) -> Net-(J26-Pin_1)
- J26 pad 2: Net-(Q38-C) -> Net-(J26-Pin_2)
- J27 pad 1: Net-(Q40-C) -> Net-(J27-Pin_1)
- J27 pad 2: Net-(Q41-C) -> Net-(J27-Pin_2)
- J28 pad 1: Net-(Q43-C) -> Net-(J28-Pin_1)
- J28 pad 2: Net-(Q44-C) -> Net-(J28-Pin_2)
- J29 pad 1: Net-(J29-Pad1) -> Net-(J29-Pin_1)
- J29 pad 2: GNDREF -> Net-(J29-Pin_2)
- J3 pad 1: Net-(J3-Pad1) -> Net-(J3-Pin_1)
- J3 pad 2: GNDREF -> Net-(J3-Pin_2)
- J30 pad 1: Net-(J30-Pad1) -> Net-(J30-Pin_1)
- J30 pad 2: GNDREF -> Net-(J30-Pin_2)
- J31 pad 1: Net-(J31-Pad1) -> Net-(J31-Pin_1)
- J31 pad 2: GNDREF -> Net-(J31-Pin_2)
- J32 pad 1: Net-(J32-Pad1) -> Net-(J32-Pin_1)
- J32 pad 2: GNDREF -> Net-(J32-Pin_2)
- J33 pad 1: Net-(J33-Pad1) -> Net-(J33-Pin_1)
- J33 pad 2: GNDREF -> Net-(J33-Pin_2)
- J34 pad 1: Net-(J34-Pad1) -> Net-(J34-Pin_1)
- J34 pad 2: GNDREF -> Net-(J34-Pin_2)
- J35 pad 1: Net-(Q52-C) -> Net-(J35-Pin_1)
- J35 pad 2: Net-(Q53-C) -> Net-(J35-Pin_2)
- J35 pad 3: Net-(Q54-C) -> Net-(J35-Pin_3)
- J36 pad 1: Net-(Q55-C) -> Net-(J36-Pin_1)
- J36 pad 2: Net-(Q56-C) -> Net-(J36-Pin_2)
- J36 pad 3: Net-(Q57-C) -> Net-(J36-Pin_3)
- J37 pad 1: Net-(Q58-C) -> Net-(J37-Pin_1)
- J37 pad 2: Net-(Q59-C) -> Net-(J37-Pin_2)
- J37 pad 3: Net-(Q60-C) -> Net-(J37-Pin_3)
- J38 pad 1: Net-(J38-Pad1) -> Net-(J38-Pin_1)
- J38 pad 2: GNDREF -> Net-(J38-Pin_2)
- J39 pad 1: Net-(J39-Pad1) -> Net-(J39-Pin_1)
- J39 pad 2: GNDREF -> Net-(J39-Pin_2)
- J4 pad 1: Net-(J4-Pad1) -> Net-(J4-Pin_1)
- J4 pad 2: GNDREF -> Net-(J4-Pin_2)
- J40 pad 1: Net-(J40-Pad1) -> Net-(J40-Pin_1)
- J40 pad 2: GNDREF -> Net-(J40-Pin_2)
- J41 pad 1: Net-(J41-Pad1) -> Net-(J41-Pin_1)
- J41 pad 2: GNDREF -> Net-(J41-Pin_2)
- J42 pad 1: Net-(J42-Pad1) -> Net-(J42-Pin_1)
- J42 pad 2: GNDREF -> Net-(J42-Pin_2)
- J43 pad 1: Net-(J43-Pad1) -> Net-(J43-Pin_1)
- J43 pad 2: GNDREF -> Net-(J43-Pin_2)
- J44 pad 1: Net-(Q67-C) -> Net-(J44-Pin_1)
- J44 pad 2: Net-(Q68-C) -> Net-(J44-Pin_2)
- J44 pad 3: Net-(Q69-C) -> Net-(J44-Pin_3)
- J45 pad 1: Net-(Q70-C) -> Net-(J45-Pin_1)
- J45 pad 2: Net-(Q71-C) -> Net-(J45-Pin_2)
- J45 pad 3: Net-(Q72-C) -> Net-(J45-Pin_3)
- J46 pad 1: Net-(Q73-C) -> /SDA
- J46 pad 2: Net-(Q74-C) -> /SCL
- J5 pad 1: Net-(J5-Pad1) -> Net-(J5-Pin_1)
- J5 pad 2: GNDREF -> Net-(J5-Pin_2)
- J6 pad 1: Net-(J6-Pad1) -> Net-(J6-Pin_1)
- J6 pad 2: GNDREF -> Net-(J6-Pin_2)
- J7 pad 1: Net-(J7-Pad1) -> Net-(J7-Pin_1)
- J7 pad 2: GNDREF -> Net-(J7-Pin_2)
- J8 pad 1: Net-(Q1-C) -> Net-(J8-Pin_1)
- J8 pad 2: Net-(Q2-C) -> Net-(J8-Pin_2)
- J9 pad 1: Net-(Q4-C) -> Net-(J9-Pin_1)
- J9 pad 2: Net-(Q5-C) -> Net-(J9-Pin_2)
- Q1 pad 1: /Cloud_Control_R1 -> Net-(J1-Pin_2)
- Q1 pad 2: Net-(Q1-C) -> /Star_Control_1
- Q1 pad 3: GNDREF -> GND
- Q10 pad 1: +5V -> Net-(J10-Pin_2)
- Q10 pad 2: /Star_Control_1 -> /Star_Control_10
- Q10 pad 3: Net-(Q10-C) -> GND
- Q11 pad 1: +5V -> Net-(J11-Pin_2)
- Q11 pad 2: /Star_Control_6 -> /Star_Control_11
- Q11 pad 3: Net-(Q11-C) -> GND
- Q12 pad 1: +5V -> Net-(J12-Pin_2)
- Q12 pad 2: /Star_Control_11 -> /Star_Control_12
- Q12 pad 3: Net-(Q12-C) -> GND
- Q13 pad 1: +5V -> Net-(J13-Pin_2)
- Q13 pad 2: /Star_Control_16 -> /Star_Control_13
- Q13 pad 3: Net-(Q13-C) -> GND
- Q14 pad 1: +5V -> Net-(J14-Pin_2)
- Q14 pad 2: /Star_Control_21 -> /Star_Control_14
- Q14 pad 3: Net-(Q14-C) -> GND
- Q15 pad 1: +5V -> Net-(J15-Pin_2)
- Q15 pad 2: /Star_Control_26 -> /Star_Control_15
- Q15 pad 3: Net-(Q15-C) -> GND
- Q16 pad 1: /Cloud_Control_R2 -> Net-(J16-Pin_2)
- Q16 pad 2: Net-(Q16-C) -> /Star_Control_16
- Q16 pad 3: GNDREF -> GND
- Q17 pad 1: /Cloud_Control_G2 -> Net-(J17-Pin_2)
- Q17 pad 2: Net-(Q17-C) -> /Star_Control_17
- Q17 pad 3: GNDREF -> GND
- Q18 pad 1: /Cloud_Control_B2 -> Net-(J18-Pin_2)
- Q18 pad 2: Net-(Q18-C) -> /Star_Control_18
- Q18 pad 3: GNDREF -> GND
- Q19 pad 1: /Cloud_Control_R2 -> Net-(J19-Pin_2)
- Q19 pad 2: Net-(Q19-C) -> /Star_Control_19
- Q19 pad 3: GNDREF -> GND
- Q2 pad 1: /Cloud_Control_G1 -> Net-(J2-Pin_2)
- Q2 pad 2: Net-(Q2-C) -> /Star_Control_2
- Q2 pad 3: GNDREF -> GND
- Q20 pad 1: /Cloud_Control_G2 -> Net-(J20-Pin_2)
- Q20 pad 2: Net-(Q20-C) -> /Star_Control_20
- Q20 pad 3: GNDREF -> GND
- Q21 pad 1: /Cloud_Control_B2 -> Net-(J21-Pin_2)
- Q21 pad 2: Net-(Q21-C) -> /Star_Control_21
- Q21 pad 3: GNDREF -> GND
- Q22 pad 1: /Cloud_Control_R2 -> Net-(J22-Pin_2)
- Q22 pad 2: Net-(Q22-C) -> /Star_Control_22
- Q22 pad 3: GNDREF -> GND
- Q23 pad 1: /Cloud_Control_G2 -> Net-(J23-Pin_2)
- Q23 pad 2: Net-(Q23-C) -> /Star_Control_23
- Q23 pad 3: GNDREF -> GND
- Q24 pad 1: /Cloud_Control_B2 -> Net-(J24-Pin_2)
- Q24 pad 2: Net-(Q24-C) -> /Star_Control_24
- Q24 pad 3: GNDREF -> GND
- Q25 pad 1: +5V -> Net-(J25-Pin_2)
- Q25 pad 2: /Star_Control_2 -> /Star_Control_25
- Q25 pad 3: Net-(Q25-C) -> GND
- Q26 pad 1: +5V -> Net-(J26-Pin_2)
- Q26 pad 2: /Star_Control_7 -> /Star_Control_26
- Q26 pad 3: Net-(Q26-C) -> GND
- Q27 pad 1: +5V -> Net-(J27-Pin_2)
- Q27 pad 2: /Star_Control_12 -> /Star_Control_27
- Q27 pad 3: Net-(Q27-C) -> GND
- Q28 pad 1: +5V -> Net-(J28-Pin_2)
- Q28 pad 2: /Star_Control_17 -> /Star_Control_28
- Q28 pad 3: Net-(Q28-C) -> GND
- Q29 pad 1: +5V -> Net-(J29-Pin_2)
- Q29 pad 2: /Star_Control_22 -> /Star_Control_29
- Q29 pad 3: Net-(Q29-C) -> GND
- Q3 pad 1: /Cloud_Control_B1 -> Net-(J3-Pin_2)
- Q3 pad 2: Net-(Q3-C) -> /Star_Control_3
- Q3 pad 3: GNDREF -> GND
- Q30 pad 1: +5V -> Net-(J30-Pin_2)
- Q30 pad 2: /Star_Control_27 -> /Star_Control_30
- Q30 pad 3: Net-(Q30-C) -> GND
- Q31 pad 1: +5V -> Net-(J31-Pin_1)
- Q31 pad 2: /Star_Control_3 -> /Cloud_Control_R5
- Q31 pad 3: Net-(Q31-C) -> GND
- Q32 pad 1: +5V -> Net-(J32-Pin_1)
- Q32 pad 2: /Star_Control_8 -> /Cloud_Control_R1
- Q32 pad 3: Net-(Q32-C) -> GND
- Q33 pad 1: +5V -> Net-(J33-Pin_1)
- Q33 pad 2: /Star_Control_13 -> /Cloud_Control_R2
- Q33 pad 3: Net-(Q33-C) -> GND
- Q34 pad 1: +5V -> Net-(J34-Pin_1)
- Q34 pad 2: /Star_Control_18 -> /Cloud_Control_R3
- Q34 pad 3: Net-(Q34-C) -> GND
- Q35 pad 1: +5V -> Net-(J35-Pin_1)
- Q35 pad 2: /Star_Control_23 -> /Cloud_Control_R4
- Q35 pad 3: Net-(Q35-C) -> GND
- Q36 pad 1: +5V -> Net-(J31-Pin_2)
- Q36 pad 2: /Star_Control_28 -> /Cloud_Control_G5
- Q36 pad 3: Net-(Q36-C) -> GND
- Q37 pad 1: /Cloud_Control_R3 -> Net-(J32-Pin_2)
- Q37 pad 2: Net-(Q37-C) -> /Cloud_Control_G1
- Q37 pad 3: GNDREF -> GND
- Q38 pad 1: /Cloud_Control_G3 -> Net-(J33-Pin_2)
- Q38 pad 2: Net-(Q38-C) -> /Cloud_Control_G2
- Q38 pad 3: GNDREF -> GND
- Q39 pad 1: /Cloud_Control_B3 -> Net-(J34-Pin_2)
- Q39 pad 2: Net-(Q39-C) -> /Cloud_Control_G3
- Q39 pad 3: GNDREF -> GND
- Q4 pad 1: /Cloud_Control_R1 -> Net-(J4-Pin_2)
- Q4 pad 2: Net-(Q4-C) -> /Star_Control_4
- Q4 pad 3: GNDREF -> GND
- Q40 pad 1: /Cloud_Control_R3 -> Net-(J35-Pin_2)
- Q40 pad 2: Net-(Q40-C) -> /Cloud_Control_G4
- Q40 pad 3: GNDREF -> GND
- Q41 pad 1: /Cloud_Control_G3 -> Net-(J31-Pin_3)
- Q41 pad 2: Net-(Q41-C) -> /Cloud_Control_B5
- Q41 pad 3: GNDREF -> GND
- Q42 pad 1: /Cloud_Control_B3 -> Net-(J32-Pin_3)
- Q42 pad 2: Net-(Q42-C) -> /Cloud_Control_B1
- Q42 pad 3: GNDREF -> GND
- Q43 pad 1: /Cloud_Control_R3 -> Net-(J33-Pin_3)
- Q43 pad 2: Net-(Q43-C) -> /Cloud_Control_B2
- Q43 pad 3: GNDREF -> GND
- Q44 pad 1: /Cloud_Control_G3 -> Net-(J34-Pin_3)
- Q44 pad 2: Net-(Q44-C) -> /Cloud_Control_B3
- Q44 pad 3: GNDREF -> GND
- Q45 pad 1: /Cloud_Control_B3 -> Net-(J35-Pin_3)
- Q45 pad 2: Net-(Q45-C) -> /Cloud_Control_B4
- Q45 pad 3: GNDREF -> GND
- Q46 pad 1: +5V -> Net-(J36-Pin_1)
- Q46 pad 2: /Star_Control_4 -> /Cloud_Control_R5
- Q46 pad 3: Net-(Q46-C) -> GND
- Q47 pad 1: +5V -> Net-(J37-Pin_1)
- Q47 pad 2: /Star_Control_9 -> /Cloud_Control_R1
- Q47 pad 3: Net-(Q47-C) -> GND
- Q48 pad 1: +5V -> Net-(J38-Pin_1)
- Q48 pad 2: /Star_Control_14 -> /Cloud_Control_R2
- Q48 pad 3: Net-(Q48-C) -> GND
- Q49 pad 1: +5V -> Net-(J39-Pin_1)
- Q49 pad 2: /Star_Control_19 -> /Cloud_Control_R3
- Q49 pad 3: Net-(Q49-C) -> GND
- Q5 pad 1: /Cloud_Control_G1 -> Net-(J5-Pin_2)
- Q5 pad 2: Net-(Q5-C) -> /Star_Control_5
- Q5 pad 3: GNDREF -> GND
- Q50 pad 1: +5V -> Net-(J40-Pin_1)
- Q50 pad 2: /Star_Control_24 -> /Cloud_Control_R4
- Q50 pad 3: Net-(Q50-C) -> GND
- Q51 pad 1: +5V -> Net-(J36-Pin_2)
- Q51 pad 2: /Star_Control_29 -> /Cloud_Control_G5
- Q51 pad 3: Net-(Q51-C) -> GND
- Q52 pad 1: /Cloud_Control_R4 -> Net-(J37-Pin_2)
- Q52 pad 2: Net-(Q52-C) -> /Cloud_Control_G1
- Q52 pad 3: GNDREF -> GND
- Q53 pad 1: /Cloud_Control_G4 -> Net-(J38-Pin_2)
- Q53 pad 2: Net-(Q53-C) -> /Cloud_Control_G2
- Q53 pad 3: GNDREF -> GND
- Q54 pad 1: /Cloud_Control_B4 -> Net-(J39-Pin_2)
- Q54 pad 2: Net-(Q54-C) -> /Cloud_Control_G3
- Q54 pad 3: GNDREF -> GND
- Q55 pad 1: /Cloud_Control_R4 -> Net-(J40-Pin_2)
- Q55 pad 2: Net-(Q55-C) -> /Cloud_Control_G4
- Q55 pad 3: GNDREF -> GND
- Q56 pad 1: /Cloud_Control_G4 -> Net-(J36-Pin_3)
- Q56 pad 2: Net-(Q56-C) -> /Cloud_Control_B5
- Q56 pad 3: GNDREF -> GND
- Q57 pad 1: /Cloud_Control_B4 -> Net-(J37-Pin_3)
- Q57 pad 2: Net-(Q57-C) -> /Cloud_Control_B1
- Q57 pad 3: GNDREF -> GND
- Q58 pad 1: /Cloud_Control_R4 -> Net-(J38-Pin_3)
- Q58 pad 2: Net-(Q58-C) -> /Cloud_Control_B2
- Q58 pad 3: GNDREF -> GND
- Q59 pad 1: /Cloud_Control_G4 -> Net-(J39-Pin_3)
- Q59 pad 2: Net-(Q59-C) -> /Cloud_Control_B3
- Q59 pad 3: GNDREF -> GND
- Q6 pad 1: /Cloud_Control_B1 -> Net-(J6-Pin_2)
- Q6 pad 2: Net-(Q6-C) -> /Star_Control_6
- Q6 pad 3: GNDREF -> GND
- Q60 pad 1: /Cloud_Control_B4 -> Net-(J40-Pin_3)
- Q60 pad 2: Net-(Q60-C) -> /Cloud_Control_B4
- Q60 pad 3: GNDREF -> GND
- Q61 pad 1: +5V -> Net-(J41-Pin_1)
- Q61 pad 2: /Star_Control_5 -> /Cloud_Control_R5
- Q61 pad 3: Net-(Q61-C) -> GND
- Q62 pad 1: +5V -> Net-(J42-Pin_1)
- Q62 pad 2: /Star_Control_10 -> /Cloud_Control_R1
- Q62 pad 3: Net-(Q62-C) -> GND
- Q63 pad 1: +5V -> Net-(J43-Pin_1)
- Q63 pad 2: /Star_Control_15 -> /Cloud_Control_R2
- Q63 pad 3: Net-(Q63-C) -> GND
- Q64 pad 1: +5V -> Net-(J44-Pin_1)
- Q64 pad 2: /Star_Control_20 -> /Cloud_Control_R3
- Q64 pad 3: Net-(Q64-C) -> GND
- Q65 pad 1: +5V -> Net-(J45-Pin_1)
- Q65 pad 2: /Star_Control_25 -> /Cloud_Control_R4
- Q65 pad 3: Net-(Q65-C) -> GND
- Q66 pad 1: +5V -> Net-(J41-Pin_2)
- Q66 pad 2: /Star_Control_30 -> /Cloud_Control_G5
- Q66 pad 3: Net-(Q66-C) -> GND
- Q67 pad 1: /Cloud_Control_R5 -> Net-(J42-Pin_2)
- Q67 pad 2: Net-(Q67-C) -> /Cloud_Control_G1
- Q67 pad 3: GNDREF -> GND
- Q68 pad 1: /Cloud_Control_G5 -> Net-(J43-Pin_2)
- Q68 pad 2: Net-(Q68-C) -> /Cloud_Control_G2
- Q68 pad 3: GNDREF -> GND
- Q69 pad 1: /Cloud_Control_B5 -> Net-(J44-Pin_2)
- Q69 pad 2: Net-(Q69-C) -> /Cloud_Control_G3
- Q69 pad 3: GNDREF -> GND
- Q7 pad 1: /Cloud_Control_R1 -> Net-(J7-Pin_2)
- Q7 pad 2: Net-(Q7-C) -> /Star_Control_7
- Q7 pad 3: GNDREF -> GND
- Q70 pad 1: /Cloud_Control_R5 -> Net-(J45-Pin_2)
- Q70 pad 2: Net-(Q70-C) -> /Cloud_Control_G4
- Q70 pad 3: GNDREF -> GND
- Q71 pad 1: /Cloud_Control_G5 -> Net-(J41-Pin_3)
- Q71 pad 2: Net-(Q71-C) -> /Cloud_Control_B5
- Q71 pad 3: GNDREF -> GND
- Q72 pad 1: /Cloud_Control_B5 -> Net-(J42-Pin_3)
- Q72 pad 2: Net-(Q72-C) -> /Cloud_Control_B1
- Q72 pad 3: GNDREF -> GND
- Q73 pad 1: /Cloud_Control_R5 -> Net-(J43-Pin_3)
- Q73 pad 2: Net-(Q73-C) -> /Cloud_Control_B2
- Q73 pad 3: GNDREF -> GND
- Q74 pad 1: /Cloud_Control_G5 -> Net-(J44-Pin_3)
- Q74 pad 2: Net-(Q74-C) -> /Cloud_Control_B3
- Q74 pad 3: GNDREF -> GND
- Q75 pad 1: /Cloud_Control_B5 -> Net-(J45-Pin_3)
- Q75 pad 2: Net-(Q75-C) -> /Cloud_Control_B4
- Q75 pad 3: GNDREF -> GND
- Q8 pad 1: /Cloud_Control_G1 -> Net-(J8-Pin_2)
- Q8 pad 2: Net-(Q8-C) -> /Star_Control_8
- Q8 pad 3: GNDREF -> GND
- Q9 pad 1: /Cloud_Control_B1 -> Net-(J9-Pin_2)
- Q9 pad 2: Net-(Q9-C) -> /Star_Control_9
- Q9 pad 3: GNDREF -> GND
- R1 pad 1: Net-(Q10-C) -> +5V
- R1 pad 2: Net-(J2-Pad1) -> Net-(J1-Pin_1)
- R10 pad 1: Net-(Q28-C) -> +5V
- R10 pad 2: Net-(J14-Pad1) -> Net-(J10-Pin_1)
- R11 pad 1: Net-(Q29-C) -> +5V
- R11 pad 2: Net-(J15-Pad1) -> Net-(J11-Pin_1)
- R12 pad 1: Net-(Q30-C) -> +5V
- R12 pad 2: Net-(J16-Pad1) -> Net-(J12-Pin_1)
- R13 pad 1: Net-(Q31-C) -> +5V
- R13 pad 2: Net-(J20-Pad1) -> Net-(J13-Pin_1)
- R14 pad 1: Net-(Q32-C) -> +5V
- R14 pad 2: Net-(J21-Pad1) -> Net-(J14-Pin_1)
- R15 pad 1: Net-(Q33-C) -> +5V
- R15 pad 2: Net-(J22-Pad1) -> Net-(J15-Pin_1)
- R16 pad 1: Net-(Q34-C) -> +5V
- R16 pad 2: Net-(J23-Pad1) -> Net-(J16-Pin_1)
- R17 pad 1: Net-(Q35-C) -> +5V
- R17 pad 2: Net-(J24-Pad1) -> Net-(J17-Pin_1)
- R18 pad 1: Net-(Q36-C) -> +5V
- R18 pad 2: Net-(J25-Pad1) -> Net-(J18-Pin_1)
- R19 pad 1: Net-(Q46-C) -> +5V
- R19 pad 2: Net-(J29-Pad1) -> Net-(J19-Pin_1)
- R2 pad 1: Net-(Q11-C) -> +5V
- R2 pad 2: Net-(J3-Pad1) -> Net-(J2-Pin_1)
- R20 pad 1: Net-(Q47-C) -> +5V
- R20 pad 2: Net-(J30-Pad1) -> Net-(J20-Pin_1)
- R21 pad 1: Net-(Q48-C) -> +5V
- R21 pad 2: Net-(J31-Pad1) -> Net-(J21-Pin_1)
- R22 pad 1: Net-(Q49-C) -> +5V
- R22 pad 2: Net-(J32-Pad1) -> Net-(J22-Pin_1)
- R23 pad 1: Net-(Q50-C) -> +5V
- R23 pad 2: Net-(J33-Pad1) -> Net-(J23-Pin_1)
- R24 pad 1: Net-(Q51-C) -> +5V
- R24 pad 2: Net-(J34-Pad1) -> Net-(J24-Pin_1)
- R25 pad 1: Net-(Q61-C) -> +5V
- R25 pad 2: Net-(J38-Pad1) -> Net-(J25-Pin_1)
- R26 pad 1: Net-(Q62-C) -> +5V
- R26 pad 2: Net-(J39-Pad1) -> Net-(J26-Pin_1)
- R27 pad 1: Net-(Q63-C) -> +5V
- R27 pad 2: Net-(J40-Pad1) -> Net-(J27-Pin_1)
- R28 pad 1: Net-(Q64-C) -> +5V
- R28 pad 2: Net-(J41-Pad1) -> Net-(J28-Pin_1)
- R29 pad 1: Net-(Q65-C) -> +5V
- R29 pad 2: Net-(J42-Pad1) -> Net-(J29-Pin_1)
- R3 pad 1: Net-(Q12-C) -> +5V
- R3 pad 2: Net-(J4-Pad1) -> Net-(J3-Pin_1)
- R30 pad 1: Net-(Q66-C) -> +5V
- R30 pad 2: Net-(J43-Pad1) -> Net-(J30-Pin_1)
- R4 pad 1: Net-(Q13-C) -> +5V
- R4 pad 2: Net-(J5-Pad1) -> Net-(J4-Pin_1)
- R5 pad 1: Net-(Q14-C) -> +5V
- R5 pad 2: Net-(J6-Pad1) -> Net-(J5-Pin_1)
- R6 pad 1: Net-(Q15-C) -> +5V
- R6 pad 2: Net-(J7-Pad1) -> Net-(J6-Pin_1)
- R7 pad 1: Net-(Q25-C) -> +5V
- R7 pad 2: Net-(J11-Pad1) -> Net-(J7-Pin_1)
- R8 pad 1: Net-(Q26-C) -> +5V
- R8 pad 2: Net-(J12-Pad1) -> Net-(J8-Pin_1)
- R9 pad 1: Net-(Q27-C) -> +5V
- R9 pad 2: Net-(J13-Pad1) -> Net-(J9-Pin_1)
- U1 pad 1: +3.3V -> GND
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Other:
- board outline added: 248.9 x 147.3 mm

Commit message: before I run the autoroute4
Parts:
- added H1: MountingHole_Pad, MountingHole:MountingHole_4.3mm_M4_DIN965_Pad_TopBottom, F.Cu at (124.5, 22.9)
- added H2: MountingHole_Pad, MountingHole:MountingHole_4.3mm_M4_DIN965_Pad_TopBottom, F.Cu at (302.3, 22.9)
- added H3: MountingHole_Pad, MountingHole:MountingHole_4.3mm_M4_DIN965_Pad_TopBottom, F.Cu at (302.3, 200.7)
- added H4: MountingHole_Pad, MountingHole:MountingHole_4.3mm_M4_DIN965_Pad_TopBottom, F.Cu at (124.5, 200.7)
- added J51: Screw_Terminal_01x02, TerminalBlock:TerminalBlock_bornier-2_P5.08mm, F.Cu at (137.2, 134.6)
- C1, C2, C3, C4, C5, C6: footprint Capacitor_SMD:C_0201_0603Metric_Pad0.64x0.40mm_HandSolder -> Capacitor_SMD:C_1206_3216Metric_Pad1.33x1.80mm_HandSolder
- J46, J47, J48, J50: footprint Library:MAX_MX126-5.0-02P-GN01-Cu-S-A -> Connector_PinHeader_2.54mm:PinHeader_1x02_P2.54mm_Vertical
- J49: value Conn_01x03 -> Screw_Terminal_01x02; footprint Library:Cixi_Kefa_Elec_KF135T-10.16-3P -> TerminalBlock:TerminalBlock_bornier-2_P5.08mm
- Q1, Q10, Q11, Q12, Q13, Q14, Q15, Q16, Q17, Q18, Q19, Q2, Q20, Q21, Q22, Q23, Q24, Q25, Q26, Q27, Q28, Q29, Q3, Q30, Q31, Q32, Q33, Q34, Q35, Q36, Q37, Q38, Q39, Q4, Q40, Q41, Q42, Q43, Q44, Q45, Q46, Q47, Q48, Q49, Q5, Q50, Q51, Q52, Q53, Q54, Q55, Q56, Q57, Q58, Q59, Q6, Q60, Q61, Q62, Q63, Q64, Q65, Q66, Q67, Q68, Q69, Q7, Q70, Q71, Q72, Q73, Q74, Q75, Q8, Q9: footprint Package_TO_SOT_THT:TO-92_Inline -> Package_TO_SOT_THT:TO-92S_Wide
- R1, R10, R11, R12, R13, R14, R15, R16, R17, R18, R19, R2, R20, R21, R22, R23, R24, R25, R26, R27, R28, R29, R3, R30, R31, R32, R33, R34, R35, R4, R5, R6, R7, R8, R9: footprint Resistor_SMD:R_0201_0603Metric_Pad0.64x0.40mm_HandSolder -> Resistor_SMD:R_1206_3216Metric_Pad1.30x1.75mm_HandSolder
- moved Q45 230.2 mm to (289.6, 193.0), turned to 90 degrees
- moved Q35 223.8 mm to (279.4, 193.0), turned to 90 degrees
- moved Q40 212.7 mm to (284.5, 193.0), turned to 90 degrees
- moved Q34 207.6 mm to (254.0, 193.0), turned to 90 degrees
- moved Q21 200.2 mm to (284.5, 94.0), turned to -90 degrees
- moved Q60 199.3 mm to (289.6, 167.6), turned to 90 degrees
- moved Q39 193.9 mm to (259.1, 193.0), turned to 90 degrees
- moved Q50 193.5 mm to (279.4, 167.6), turned to 90 degrees
- moved Q55 187.9 mm to (284.5, 167.6), turned to 90 degrees
- moved Q22 185.5 mm to (269.2, 94.0), turned to -90 degrees
- moved Q44 184.0 mm to (264.2, 193.0), turned to 90 degrees
- moved J35 181.2 mm to (279.5, 198.1)
- moved Q59 179.8 mm to (264.2, 167.6), turned to 90 degrees
- moved Q70 177.2 mm to (283.8, 134.6), turned to 90 degrees
- moved Q38 177.1 mm to (233.7, 193.0), turned to 90 degrees
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Connections:
- J49 pad 1: +3.3V -> +5V
- J49 pad 2: +5V -> GND
Routing:
- net +5V: track 0.00 -> 53.6 mm, vias 0 -> 30
- added copper zone on B.Cu, net +5V
- added copper zone on F.Cu, net GND
Other:
- board size 248.9 x 147.3 mm -> 188 x 188 mm
- board text added: "3V3"
- board text added: "5V0"
- board text added: "GND"
- board text added: "RX"
- board text added: "SCL"
- board text added: "SDA"
- board text added: "TX"

Commit message: main2: ERC Check
Changed lines of the file:
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@@
   (gr_rect (start 119.38 17.78) (end 307.34 205.74)
     (stroke (width 0.1) (type default)) (fill none) (layer "Edge.Cuts"))
-  (gr_rect (start 119.38 205.74) (end 307.34 17.78)
+  (gr_rect (start 119.38 17.78) (end 307.34 205.74)
     (stroke (width 0.1) (type default)) (fill none) (layer "Edge.Cuts"))
   (gr_text "5V0" (at 129.54 182.88) (layer "F.SilkS")

Commit message: main2: Manual routing
Routing:
- net +3.3V: track 0.00 -> 109.0 mm
Changed lines of the file:
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@@
     (effects (font (size 1.5 1.5) (thickness 0.3) bold))
   )
+  (segment (start 137.16 134.62) (end 146.735 134.62) (width 1) (layer "F.Cu") (net 1))
+  (segment (start 149.007008 134.035) (end 149.726004 134.753996) (width 1) (layer "F.Cu") (net 1))
+  (segment (start 149.726004 134.753996) (end 149.726004 188.093996) (width 1) (layer "F.Cu") (net 1))
+  (segment (start 147.32 134.035) (end 149.007008 134.035) (width 1) (layer "F.Cu") (net 1))
+  (segment (start 146.735 134.62) (end 147.32 134.035) (width 1) (layer "F.Cu") (net 1))
+  (segment (start 134.62 193.04) (end 144.78 193.04) (width 1) (layer "F.Cu") (net 1))
+  (segment (start 149.726004 188.093996) (end 144.78 193.04) (width 1) (layer "F.Cu") (net 1))
+  (segment (start 144.78 193.04) (end 170.18 193.04) (width 1) (layer "F.Cu") (net 1))
   (segment (start 152.4 69.36) (end 152.4 71.12) (width 1) (layer "F.Cu") (net 5))
   (segment (start 182.88 69.36) (end 182.88 71.12) (width 1) (layer "F.Cu") (net 5))

Commit message: main2: All done :)
Routing:
- net +3.3V: track 109.0 -> 467.1 mm, vias 0 -> 5
- net /SCL: track 0.00 -> 343.4 mm, vias 0 -> 2
- net /SDA: track 0.00 -> 241.1 mm, vias 0 -> 3
- net GND: track 0.00 -> 178.0 mm, vias 0 -> 14
- net /Cloud_Control_R5: track 0.00 -> 148.6 mm
- net /Cloud_Control_B5: track 0.00 -> 141.0 mm
- net /Cloud_Control_G5: track 0.00 -> 132.3 mm, vias 0 -> 2
- net /Cloud_Control_G3: track 0.00 -> 123.0 mm, vias 0 -> 1
- net /Cloud_Control_B4: track 0.00 -> 119.4 mm
- net /Cloud_Control_B3: track 0.00 -> 114.7 mm, vias 0 -> 2
- net /Cloud_Control_G4: track 0.00 -> 113.9 mm
- net /Cloud_Control_R4: track 0.00 -> 110.3 mm, vias 0 -> 2
- net /Star_Control_20: track 0.00 -> 98.5 mm, vias 0 -> 2
- net /Cloud_Control_R1: track 0.00 -> 97.6 mm
- net /Star_Control_21: track 0.00 -> 95.8 mm, vias 0 -> 2
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
Commit message: DONE! (v3)
Other:
- board text added: "GNCTR PCB Cloud and Star Control"
