File: Cloud-Star-Lights-PCB/Cloud-Star-Lights-PCB.kicad_pcb (KiCad board)
At the start: 2 copper layers, 188 x 188 mm, 175 parts, among them J1 Conn_01x02, J10 Conn_01x02, J11 Conn_01x02, J12 Conn_01x02, J13 Conn_01x02, J14 Conn_01x02, J15 Conn_01x02, J16 Conn_01x02, J17 Conn_01x02, J18 Conn_01x02, J19 Conn_01x02, J2 Conn_01x02, J20 Conn_01x02, J21 Conn_01x02, J22 Conn_01x02, J23 Conn_01x02, J24 Conn_01x02, J25 Conn_01x02, J26 Conn_01x02, J27 Conn_01x02, J28 Conn_01x02, J29 Conn_01x02, J3 Conn_01x02, J30 Conn_01x02, J31 Conn_01x04, J32 Conn_01x04, J33 Conn_01x04, J34 Conn_01x04, J35 Conn_01x04, J36 Conn_01x04, J37 Conn_01x04, J38 Conn_01x04, J39 Conn_01x04, J4 Conn_01x02, J40 Conn_01x04, J41 Conn_01x04, J42 Conn_01x04, J43 Conn_01x04, J44 Conn_01x04, J45 Conn_01x04, J46 Conn_01x02, J47 Conn_01x02, J48 Conn_01x02, J49 Screw_Terminal_01x02, J5 Conn_01x02, J50 Conn_01x02, J51 Screw_Terminal_01x02, J6 Conn_01x02, J7 Conn_01x02, J8 Conn_01x02, J9 Conn_01x02, Q1 2N3906, Q10 2N3906, Q11 2N3906, Q12 2N3906, Q13 2N3906, Q14 2N3906, Q15 2N3906, Q16 2N3906, Q17 2N3906, Q18 2N3906, Q19 2N3906, Q2 2N3906, Q20 2N3906, Q21 2N3906, Q22 2N3906, Q23 2N3906, Q24 2N3906, Q25 2N3906, Q26 2N3906, Q27 2N3906, Q28 2N3906, Q29 2N3906, Q3 2N3906, Q30 2N3906, Q31 2N3906, Q32 2N3906, Q33 2N3906, Q34 2N3906, Q35 2N3906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

Commit message: Starting routing
Parts:
- removed Q16, Q17, Q18, Q19, Q20, Q21, Q22, Q23, Q24, Q25, Q26, Q27, Q28, Q29, Q30, Q31, Q32, Q33, Q34, Q35, Q36, Q37, Q38, Q39, Q40, Q41, Q42, Q43, Q44, Q45, Q46, Q47, Q48, Q49, Q50, Q51, Q52, Q53, Q54, Q55, Q56, Q57, Q58, Q59, Q60, Q61, Q62, Q63, Q64, Q65, Q66, Q67, Q68, Q69, Q70, Q71, Q72, Q73, Q74, Q75: 2N3906, Package_TO_SOT_THT:TO-92S_Wide
- removed U4: PCA9635, Package_SO:TSSOP-28_4.4x9.7mm_P0.65mm
- added J52: Conn_01x04, Connector_PinHeader_2.54mm:PinHeader_1x04_P2.54mm_Vertical, F.Cu at (179.7, 111.6)
- added J53: Conn_01x04, Connector_PinHeader_2.54mm:PinHeader_1x04_P2.54mm_Vertical, F.Cu at (184.3, 111.6)
- added R36: ?kΩ, Resistor_SMD:R_1206_3216Metric_Pad1.30x1.75mm_HandSolder, F.Cu at (55.7, 92.4)
- added R37: 1kΩ, Resistor_SMD:R_1206_3216Metric_Pad1.30x1.75mm_HandSolder, F.Cu at (93.9, 84.8)
- added R38: 3.3kΩ, Resistor_SMD:R_1206_3216Metric_Pad1.30x1.75mm_HandSolder, F.Cu at (91.4, 84.8)
- added R39: 1kΩ, Resistor_SMD:R_1206_3216Metric_Pad1.30x1.75mm_HandSolder, F.Cu at (108.2, 101.8)
- added R40: 3.3kΩ, Resistor_SMD:R_1206_3216Metric_Pad1.30x1.75mm_HandSolder, F.Cu at (105.4, 101.8)
- added R41: 1kΩ, Resistor_SMD:R_1206_3216Metric_Pad1.30x1.75mm_HandSolder, F.Cu at (93.9, 110.3)
- added R42: 3.3kΩ, Resistor_SMD:R_1206_3216Metric_Pad1.30x1.75mm_HandSolder, F.Cu at (91.4, 110.3)
- added R43: 1kΩ, Resistor_SMD:R_1206_3216Metric_Pad1.30x1.75mm_HandSolder, F.Cu at (108.2, 93.3)
- added R44: 3.3kΩ, Resistor_SMD:R_1206_3216Metric_Pad1.30x1.75mm_HandSolder, F.Cu at (105.4, 93.3)
- added R45: 1kΩ, Resistor_SMD:R_1206_3216Metric_Pad1.30x1.75mm_HandSolder, F.Cu at (79.5, 93.3)
- added R46: 3.3kΩ, Resistor_SMD:R_1206_3216Metric_Pad1.30x1.75mm_HandSolder, F.Cu at (76.8, 93.3)
- added R47: 1kΩ, Resistor_SMD:R_1206_3216Metric_Pad1.30x1.75mm_HandSolder, F.Cu at (79.4, 84.8)
- added R48: 3.3kΩ, Resistor_SMD:R_1206_3216Metric_Pad1.30x1.75mm_HandSolder, F.Cu at (76.7, 84.8)
- added R49: 1kΩ, Resistor_SMD:R_1206_3216Metric_Pad1.30x1.75mm_HandSolder, F.Cu at (93.9, 101.8)
- added R50: 3.3kΩ, Resistor_SMD:R_1206_3216Metric_Pad1.30x1.75mm_HandSolder, F.Cu at (91.4, 101.8)
- added R51: 1kΩ, Resistor_SMD:R_1206_3216Metric_Pad1.30x1.75mm_HandSolder, F.Cu at (79.5, 110.3)
- added R52: 3.3kΩ, Resistor_SMD:R_1206_3216Metric_Pad1.30x1.75mm_HandSolder, F.Cu at (76.8, 110.3)
- added R53: 1kΩ, Resistor_SMD:R_1206_3216Metric_Pad1.30x1.75mm_HandSolder, F.Cu at (93.9, 93.3)
- added R54: 3.3kΩ, Resistor_SMD:R_1206_3216Metric_Pad1.30x1.75mm_HandSolder, F.Cu at (91.4, 93.3)
- added R55: 1kΩ, Resistor_SMD:R_1206_3216Metric_Pad1.30x1.75mm_HandSolder, F.Cu at (93.9, 118.8)
- added R56: 3.3kΩ, Resistor_SMD:R_1206_3216Metric_Pad1.30x1.75mm_HandSolder, F.Cu at (91.4, 118.8)
- added R57: 1kΩ, Resistor_SMD:R_1206_3216Metric_Pad1.30x1.75mm_HandSolder, F.Cu at (108.2, 118.8)
- added R58: 3.3kΩ, Resistor_SMD:R_1206_3216Metric_Pad1.30x1.75mm_HandSolder, F.Cu at (105.4, 118.8)
- added R59: 1kΩ, Resistor_SMD:R_1206_3216Metric_Pad1.30x1.75mm_HandSolder, F.Cu at (79.5, 101.8)
- added R60: 3.3kΩ, Resistor_SMD:R_1206_3216Metric_Pad1.30x1.75mm_HandSolder, F.Cu at (76.8, 101.8)
- added R61: 1kΩ, Resistor_SMD:R_1206_3216Metric_Pad1.30x1.75mm_HandSolder, F.Cu at (108.2, 110.3)
- added R62: 3.3kΩ, Resistor_SMD:R_1206_3216Metric_Pad1.30x1.75mm_HandSolder, F.Cu at (105.4, 110.3)
- added R63: 1kΩ, Resistor_SMD:R_1206_3216Metric_Pad1.30x1.75mm_HandSolder, F.Cu at (79.5, 118.8)
- added R64: 3.3kΩ, Resistor_SMD:R_1206_3216Metric_Pad1.30x1.75mm_HandSolder, F.Cu at (76.8, 118.8)
- C1, C2, C4: value 10uf -> 0.1uF; footprint Capacitor_SMD:C_1206_3216Metric_Pad1.33x1.80mm_HandSolder -> Package_TO_SOT_THT:SOD-70_P5.08mm
- J1, J10, J11, J12, J13, J14, J15, J16, J17, J18, J19, J2, J20, J21, J22, J23, J24, J25, J26, J27, J28, J29, J3, J30, J4, J5, J6, J7, J8, J9: value Conn_01x02 -> Conn_02x01; footprint Library:MAX_MX126-5.0-02P-GN01-Cu-S-A -> Connector_PinHeader_2.54mm:PinHeader_1x02_P2.54mm_Vertical
- J31, J32: value Conn_01x04 -> Conn_02x01; footprint Library:JILN_JL301-50004U01 -> Connector_PinHeader_2.54mm:PinHeader_1x02_P2.54mm_Vertical
- J33, J34, J35, J36, J37, J38, J39, J40, J41, J42, J43, J44, J45: footprint Library:JILN_JL301-50004U01 -> Connector_PinHeader_2.54mm:PinHeader_1x04_P2.54mm_Vertical
- Q1, Q10, Q11, Q12, Q13, Q14, Q15, Q2, Q3, Q4, Q5, Q6, Q7, Q8, Q9: value 2N3906 -> BS170; footprint Package_TO_SOT_THT:TO-92S_Wide -> Package_TO_SOT_THT:TO-92_Inline
- R1, R10, R11, R12, R13, R14, R15, R16, R19, R2, R20, R21, R22, R23, R24, R25, R26, R27, R28, R29, R3, R30, R4, R5, R6, R7, R8, R9: value 22Ω -> ?kΩ
- R17: value 22Ω -> 1kΩ
- R18: value 22Ω -> 3.3kΩ
- R31, R34, R35: value 10kΩ -> ?kΩ
- R32, R33: value 10kΩ -> 3.3kΩ
- U1, U3: value PCA9635 -> TLC59116FIPWR; footprint Package_SO:TSSOP-28_4.4x9.7mm_P0.65mm -> Library:TLC59116FIPWR
- moved J21 262.2 mm to (27.7, 75.9), turned to 0 degrees
- moved J1 262.0 mm to (27.9, 37.5), turned to 0 degrees
- moved R1 250.3 mm to (39.4, 38.7), turned to -90 degrees
- moved J11 245.3 mm to (44.5, 52.7), turned to 0 degrees
- moved R2 243.3 mm to (31.1, 38.7), turned to -90 degrees
- moved R21 243.2 mm to (47.4, 69.6), turned to -90 degrees
- moved R11 242.3 mm to (47.6, 54.0), turned to -90 degrees
- moved J22 238.7 mm to (36.0, 75.9), turned to 0 degrees
- moved J2 238.5 mm to (36.2, 37.5), turned to 0 degrees
- moved J13 231.2 mm to (27.9, 60.3), turned to 0 degrees
- moved R23 228.9 mm to (30.9, 77.2), turned to -90 degrees
- moved R13 228.0 mm to (31.1, 61.6), turned to -90 degrees
- moved J12 221.8 mm to (52.7, 52.7), turned to 0 degrees
- moved R22 219.9 mm to (55.7, 69.6), turned to -90 degrees
- moved R12 218.9 mm to (55.9, 54.0), turned to -90 degrees
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Connections:
- C1 pad 2: +3.3V -> Net-(U2-EN)
- C2 pad 1: GND -> +3.3V
- C2 pad 2: +3.3V -> GND
- C4 pad 1: GND -> +5V
- C4 pad 2: +3.3V -> GND
- J33 pad 1: Net-(J33-Pin_1) -> /CloudController/Output1
- J33 pad 2: Net-(J33-Pin_2) -> /CloudController/Output6
- J33 pad 3: Net-(J33-Pin_3) -> /CloudController/Output11
- J34 pad 1: Net-(J34-Pin_1) -> unconnected-(J34-Pin_1-Pad1)
- J34 pad 2: Net-(J34-Pin_2) -> unconnected-(J34-Pin_2-Pad2)
- J34 pad 3: Net-(J34-Pin_3) -> unconnected-(J34-Pin_3-Pad3)
- J34 pad 4: +5V -> unconnected-(J34-Pin_4-Pad4)
- J35 pad 1: Net-(J35-Pin_1) -> /CloudController/Output1
- J35 pad 2: Net-(J35-Pin_2) -> /CloudController/Output6
- J35 pad 3: Net-(J35-Pin_3) -> /CloudController/Output11
- J36 pad 1: Net-(J36-Pin_1) -> /CloudController/Output2
- J36 pad 2: Net-(J36-Pin_2) -> /CloudController/Output7
- J36 pad 3: Net-(J36-Pin_3) -> /CloudController/Output12
- J37 pad 1: Net-(J37-Pin_1) -> unconnected-(J37-Pin_1-Pad1)
- J37 pad 2: Net-(J37-Pin_2) -> unconnected-(J37-Pin_2-Pad2)
- J37 pad 3: Net-(J37-Pin_3) -> unconnected-(J37-Pin_3-Pad3)
- J37 pad 4: +5V -> unconnected-(J37-Pin_4-Pad4)
- J38 pad 1: Net-(J38-Pin_1) -> /CloudController/Output2
- J38 pad 2: Net-(J38-Pin_2) -> /CloudController/Output7
- J38 pad 3: Net-(J38-Pin_3) -> /CloudController/Output12
- J39 pad 1: Net-(J39-Pin_1) -> /CloudController/Output3
- J39 pad 2: Net-(J39-Pin_2) -> /CloudController/Output8
- J39 pad 3: Net-(J39-Pin_3) -> /CloudController/Output13
- J40 pad 1: Net-(J40-Pin_1) -> unconnected-(J40-Pin_1-Pad1)
- J40 pad 2: Net-(J40-Pin_2) -> unconnected-(J40-Pin_2-Pad2)
- J40 pad 3: Net-(J40-Pin_3) -> unconnected-(J40-Pin_3-Pad3)
- J40 pad 4: +5V -> unconnected-(J40-Pin_4-Pad4)
- J41 pad 1: Net-(J41-Pin_1) -> /CloudController/Output3
- J41 pad 2: Net-(J41-Pin_2) -> /CloudController/Output8
- J41 pad 3: Net-(J41-Pin_3) -> /CloudController/Output13
- J42 pad 1: Net-(J42-Pin_1) -> /CloudController/Output4
- J42 pad 2: Net-(J42-Pin_2) -> /CloudController/Output9
- J42 pad 3: Net-(J42-Pin_3) -> /CloudController/Output14
- J43 pad 1: Net-(J43-Pin_1) -> unconnected-(J43-Pin_1-Pad1)
- J43 pad 2: Net-(J43-Pin_2) -> unconnected-(J43-Pin_2-Pad2)
- J43 pad 3: Net-(J43-Pin_3) -> unconnected-(J43-Pin_3-Pad3)
- J43 pad 4: +5V -> unconnected-(J43-Pin_4-Pad4)
- J44 pad 1: Net-(J44-Pin_1) -> /CloudController/Output4
- J44 pad 2: Net-(J44-Pin_2) -> /CloudController/Output9
- J44 pad 3: Net-(J44-Pin_3) -> /CloudController/Output14
- J45 pad 1: Net-(J45-Pin_1) -> /CloudController/Output5
- J45 pad 2: Net-(J45-Pin_2) -> /CloudController/Output10
- J45 pad 3: Net-(J45-Pin_3) -> /CloudController/Output15
- Q1 pad 1: Net-(J1-Pin_2) -> /CloudController/Output2
- Q1 pad 2: /Star_Control_1 -> Net-(Q1-G)
- Q10 pad 1: Net-(J10-Pin_2) -> /CloudController/Output10
- Q10 pad 2: /Star_Control_10 -> Net-(Q10-G)
- Q11 pad 1: Net-(J11-Pin_2) -> /CloudController/Output11
- Q11 pad 2: /Star_Control_11 -> Net-(Q11-G)
- Q12 pad 1: Net-(J12-Pin_2) -> /CloudController/Output12
- Q12 pad 2: /Star_Control_12 -> Net-(Q12-G)
- Q13 pad 1: Net-(J13-Pin_2) -> /CloudController/Output13
- Q13 pad 2: /Star_Control_13 -> Net-(Q13-G)
- Q14 pad 1: Net-(J14-Pin_2) -> /CloudController/Output14
- Q14 pad 2: /Star_Control_14 -> Net-(Q14-G)
- Q15 pad 1: Net-(J15-Pin_2) -> /CloudController/Output15
- Q15 pad 2: /Star_Control_15 -> Net-(Q15-G)
- Q2 pad 1: Net-(J2-Pin_2) -> /CloudController/Output1
- Q2 pad 2: /Star_Control_2 -> Net-(Q2-G)
- Q3 pad 1: Net-(J3-Pin_2) -> /CloudController/Output3
- Q3 pad 2: /Star_Control_3 -> Net-(Q3-G)
- Q4 pad 1: Net-(J4-Pin_2) -> /CloudController/Output4
- Q4 pad 2: /Star_Control_4 -> Net-(Q4-G)
- Q5 pad 1: Net-(J5-Pin_2) -> /CloudController/Output5
- Q5 pad 2: /Star_Control_5 -> Net-(Q5-G)
- Q6 pad 1: Net-(J6-Pin_2) -> /CloudController/Output6
- Q6 pad 2: /Star_Control_6 -> Net-(Q6-G)
- Q7 pad 1: Net-(J7-Pin_2) -> /CloudController/Output7
- Q7 pad 2: /Star_Control_7 -> Net-(Q7-G)
- Q8 pad 1: Net-(J8-Pin_2) -> /CloudController/Output8
- Q8 pad 2: /Star_Control_8 -> Net-(Q8-G)
- Q9 pad 1: Net-(J9-Pin_2) -> /CloudController/Output9
- Q9 pad 2: /Star_Control_9 -> Net-(Q9-G)
- R1 pad 2: Net-(J1-Pin_1) -> Net-(J2-Pin_2)
- R10 pad 2: Net-(J10-Pin_1) -> Net-(J10-Pin_2)
- R11 pad 2: Net-(J11-Pin_1) -> Net-(J11-Pin_2)
- R12 pad 2: Net-(J12-Pin_1) -> Net-(J12-Pin_2)
- R13 pad 2: Net-(J13-Pin_1) -> Net-(J13-Pin_2)
- R14 pad 2: Net-(J14-Pin_1) -> Net-(J14-Pin_2)
- R15 pad 2: Net-(J15-Pin_1) -> Net-(J15-Pin_2)
- R16 pad 2: Net-(J16-Pin_1) -> Net-(J16-Pin_2)
- R17 pad 1: +5V -> /Control2
- R17 pad 2: Net-(J17-Pin_1) -> Net-(Q1-G)
- R18 pad 1: +5V -> Net-(Q1-G)
- R18 pad 2: Net-(J18-Pin_1) -> GND
- R19 pad 2: Net-(J19-Pin_1) -> Net-(J17-Pin_2)
- R2 pad 2: Net-(J2-Pin_1) -> Net-(J1-Pin_2)
- R20 pad 2: Net-(J20-Pin_1) -> Net-(J18-Pin_2)
- R21 pad 2: Net-(J21-Pin_1) -> Net-(J19-Pin_2)
- R22 pad 2: Net-(J22-Pin_1) -> Net-(J20-Pin_2)
- R23 pad 2: Net-(J23-Pin_1) -> Net-(J21-Pin_2)
- R24 pad 2: Net-(J24-Pin_1) -> Net-(J22-Pin_2)
- R25 pad 2: Net-(J25-Pin_1) -> Net-(J23-Pin_2)
- R26 pad 2: Net-(J26-Pin_1) -> Net-(J24-Pin_2)
- R27 pad 2: Net-(J27-Pin_1) -> Net-(J25-Pin_2)
- R28 pad 2: Net-(J28-Pin_1) -> Net-(J26-Pin_2)
- R29 pad 2: Net-(J29-Pin_1) -> Net-(J27-Pin_2)
- R3 pad 2: Net-(J3-Pin_1) -> Net-(J3-Pin_2)
- R30 pad 2: Net-(J30-Pin_1) -> Net-(J28-Pin_2)
- R31 pad 1: Net-(U1-~{OE}) -> +5V
- R31 pad 2: GND -> Net-(J29-Pin_2)
- R34 pad 1: Net-(U3-~{OE}) -> +5V
- R34 pad 2: GND -> Net-(J30-Pin_2)
- R35 pad 1: Net-(U4-~{OE}) -> +5V
- R35 pad 2: GND -> Net-(J31-Pin_2)
- R4 pad 2: Net-(J4-Pin_1) -> Net-(J4-Pin_2)
- R5 pad 2: Net-(J5-Pin_1) -> Net-(J5-Pin_2)
- R6 pad 2: Net-(J6-Pin_1) -> Net-(J6-Pin_2)
- R7 pad 2: Net-(J7-Pin_1) -> Net-(J7-Pin_2)
- R8 pad 2: Net-(J8-Pin_1) -> Net-(J8-Pin_2)
- R9 pad 2: Net-(J9-Pin_1) -> Net-(J9-Pin_2)
- U1 pad 1: GND -> unconnected-(U1-REXT-Pad1)
- U1 pad 10: /Star_Control_5 -> GND
- U1 pad 11: /Star_Control_6 -> Net-(J13-Pin_1)
- U1 pad 12: /Star_Control_7 -> Net-(J14-Pin_1)
- U1 pad 13: /Star_Control_8 -> Net-(J15-Pin_1)
- U1 pad 14: GND -> Net-(J16-Pin_1)
- U1 pad 15: /Star_Control_9 -> Net-(J8-Pin_1)
- U1 pad 16: /Star_Control_10 -> Net-(J7-Pin_1)
- U1 pad 17: /Star_Control_11 -> Net-(J6-Pin_1)
- U1 pad 18: /Star_Control_12 -> Net-(J5-Pin_1)
- U1 pad 19: /Star_Control_13 -> GND
- U1 pad 2: +3.3V -> GND
- U1 pad 20: /Star_Control_14 -> Net-(J4-Pin_1)
- U1 pad 21: /Star_Control_15 -> Net-(J3-Pin_1)
- U1 pad 22: unconnected-(U1-LED15-Pad22) -> Net-(J2-Pin_1)
- U1 pad 23: Net-(U1-~{OE}) -> Net-(J1-Pin_1)
- U1 pad 24: +3.3V -> GND
- U1 pad 25: +3.3V -> +5V
- U1 pad 28: +3.3V -> +5V
- U1 pad 3: +3.3V -> GND
- U1 pad 4: +3.3V -> GND
- U1 pad 5: +3.3V -> GND
- U1 pad 6: /Star_Control_1 -> Net-(J9-Pin_1)
- U1 pad 7: /Star_Control_2 -> Net-(J10-Pin_1)
- U1 pad 8: /Star_Control_3 -> Net-(J11-Pin_1)
- U1 pad 9: /Star_Control_4 -> Net-(J12-Pin_1)
- U2 pad 15: unconnected-(U2-D23/VSPI_MOSI-Pad15) -> /Control8
- U2 pad 19: unconnected-(U2-D34/ADC1_CH6-Pad19) -> /Control14
- U2 pad 20: unconnected-(U2-D35/ADC1_CH7-Pad20) -> /Control15
- U2 pad 21: unconnected-(U2-D32/ADC1_CH4/TOUCH9-Pad21) -> /Control12
- U2 pad 22: unconnected-(U2-D33/ADC1_CH5/TOUCH8-Pad22) -> /Control13
- U2 pad 23: unconnected-(U2-D25/ADC2_CH8/DAC1-Pad23) -> /Control9
- U2 pad 24: unconnected-(U2-D26/ADC2_CH9/DAC2-Pad24) -> /Control10
- U2 pad 25: unconnected-(U2-D27/ADC2_CH7/TOUCH7-Pad25) -> /Control11
- U2 pad 26: unconnected-(U2-D14/ADC2_CH6/TOUCH6/HSPI_CLK-Pad26) -> /Control6
- U2 pad 27: unconnected-(U2-D12/ADC2_CH5/TOUCH5/HSPI_MISO-Pad27) -> /Control4
- U2 pad 28: unconnected-(U2-D13/ADC2_CH4/TOUCH4/HSPI_MOSI-Pad28) -> /Control5
- U2 pad 3: unconnected-(U2-D15/ADC2_CH3/TOUCH3/HSPI_CS0-Pad3) -> /Control7
- U2 pad 30: +3.3V -> +5V
- U2 pad 4: unconnected-(U2-D2/ADC2_CH2/TOUCH2-Pad4) -> /Control1
- U2 pad 5: unconnected-(U2-D4/ADC2_CH0/TOUCH0-Pad5) -> /Control2
- U2 pad 8: unconnected-(U2-D5/VSPI_CS0-Pad8) -> /Control3
- U3 pad 1: GND -> unconnected-(U3-REXT-Pad1)
- U3 pad 10: /Star_Control_20 -> GND
- U3 pad 11: /Star_Control_21 -> Net-(J20-Pin_1)
- U3 pad 12: /Star_Control_22 -> Net-(J19-Pin_1)
- U3 pad 13: /Star_Control_23 -> Net-(J18-Pin_1)
- U3 pad 14: GND -> Net-(J17-Pin_1)
- U3 pad 15: /Star_Control_24 -> Net-(J32-Pin_1)
- U3 pad 16: /Star_Control_25 -> Net-(J31-Pin_1)
- U3 pad 17: /Star_Control_26 -> Net-(J30-Pin_1)
- U3 pad 18: /Star_Control_27 -> Net-(J29-Pin_1)
- U3 pad 19: /Star_Control_28 -> GND
- U3 pad 2: +3.3V -> +5V
- U3 pad 20: /Star_Control_29 -> Net-(J28-Pin_1)
- U3 pad 21: /Star_Control_30 -> Net-(J27-Pin_1)
- U3 pad 22: unconnected-(U3-LED15-Pad22) -> Net-(J26-Pin_1)
- U3 pad 23: Net-(U3-~{OE}) -> Net-(J25-Pin_1)
- U3 pad 24: +3.3V -> GND
- U3 pad 25: +3.3V -> +5V
- U3 pad 28: +3.3V -> +5V
- U3 pad 3: +3.3V -> GND
- U3 pad 4: +3.3V -> GND
- U3 pad 5: +3.3V -> GND
- U3 pad 6: /Star_Control_16 -> Net-(J24-Pin_1)
- U3 pad 7: /Star_Control_17 -> Net-(J23-Pin_1)
- U3 pad 8: /Star_Control_18 -> Net-(J22-Pin_1)
- U3 pad 9: /Star_Control_19 -> Net-(J21-Pin_1)
Routing:
- net +3.3V: track 467.1 -> 56.6 mm, vias 5 -> 0
- net /SCL: track 343.4 -> 12.5 mm, vias 2 -> 0
- net /SDA: track 241.1 -> 9.32 mm, vias 3 -> 0
- net GND: track 178.0 -> 0.00 mm, vias 14 -> 0
- net /Cloud_Control_R5: track 148.6 -> 0.00 mm
- net /Cloud_Control_B5: track 141.0 -> 0.00 mm
- net /Cloud_Control_G5: track 132.3 -> 0.00 mm, vias 2 -> 0
- net /Cloud_Control_G3: track 123.0 -> 0.00 mm, vias 1 -> 0
- net /Cloud_Control_B4: track 119.4 -> 0.00 mm
- net /Cloud_Control_B3: track 114.7 -> 0.00 mm, vias 2 -> 0
- net /Cloud_Control_G4: track 113.9 -> 0.00 mm
- net /Cloud_Control_R4: track 110.3 -> 0.00 mm, vias 2 -> 0
- net /Star_Control_20: track 98.5 -> 0.00 mm, vias 2 -> 0
- net /Cloud_Control_R1: track 97.6 -> 0.00 mm
- net /Star_Control_21: track 95.8 -> 0.00 mm, vias 2 -> 0
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- added copper zone on F.Cu, net +5V
- removed copper zone on B.Cu, net +5V
Other:
- board size 188 x 188 mm -> 100 x 100 mm
- board text removed: "3V3"
- board text removed: "5V0"
- board text removed: "GNCTR PCB Cloud and Star Control"
- board text removed: "GND"
- board text removed: "RX"
- board text removed: "SCL"
- board text removed: "SDA"
- board text removed: "TX"
