File: Cloud-Star-Lights-PCB/Cloud-Star-Lights-PCB.kicad_pcb (KiCad board)
At the start: 2 copper layers, 100 x 100 mm, 145 parts, among them J1 Conn_02x01, J10 Conn_02x01, J11 Conn_02x01, J12 Conn_02x01, J13 Conn_02x01, J14 Conn_02x01, J15 Conn_02x01, J16 Conn_02x01, J17 Conn_02x01, J18 Conn_02x01, J19 Conn_02x01, J2 Conn_02x01, J20 Conn_02x01, J21 Conn_02x01, J22 Conn_02x01, J23 Conn_02x01, J24 Conn_02x01, J25 Conn_02x01, J26 Conn_02x01, J27 Conn_02x01, J28 Conn_02x01, J29 Conn_02x01, J3 Conn_02x01, J30 Conn_02x01, J31 Conn_02x01, J32 Conn_02x01, J33 Conn_01x04, J34 Conn_01x04, J35 Conn_01x04, J36 Conn_01x04, J37 Conn_01x04, J38 Conn_01x04, J39 Conn_01x04, J4 Conn_02x01, J40 Conn_01x04, J41 Conn_01x04, J42 Conn_01x04, J43 Conn_01x04, J44 Conn_01x04, J45 Conn_01x04, J46 Conn_01x02, J47 Conn_01x02, J48 Conn_01x02, J49 Screw_Terminal_01x02, J5 Conn_02x01, J50 Conn_01x02, J51 Screw_Terminal_01x02, J52 Conn_01x04, J53 Conn_01x04, J6 Conn_02x01, J7 Conn_02x01, J8 Conn_02x01, J9 Conn_02x01, Q1 BS170, Q10 BS170, Q11 BS170, Q12 BS170, Q13 BS170, Q14 BS170, Q15 BS170, Q2 BS170, Q3 BS170, Q4 BS170, Q5 BS170, Q6 BS170, Q7 BS170, Q8 BS170, Q9 BS170, U1 TLC59116FIPWR, U2 ESP32-Module-30Pin, U3 TLC59116FIPWR

Commit message: Unrouted board
Parts:
- moved J38 161.7 mm to (70.5, 27.3), turned to 90 degrees
- moved J53 156.9 mm to (52.1, 27.1), turned to 90 degrees
- moved J37 155.6 mm to (70.5, 31.8), turned to 90 degrees
- moved J52 150.5 mm to (52.1, 31.8), turned to 90 degrees
- moved J36 149.5 mm to (70.5, 36.2), turned to 90 degrees
- moved J45 144.1 mm to (52.1, 36.4), turned to 90 degrees
- moved J44 119.9 mm to (87.0, 27.3), turned to 90 degrees
- moved J35 117.9 mm to (105.4, 27.3), turned to 90 degrees
- moved J43 113.5 mm to (87.0, 31.8), turned to 90 degrees
- moved J34 111.5 mm to (105.4, 31.8), turned to 90 degrees
- moved J42 107.2 mm to (87.0, 36.2), turned to 90 degrees
- moved J33 105.2 mm to (105.4, 36.2), turned to 90 degrees
- moved J41 90.8 mm to (122.1, 59.7)
- moved J39 90.8 mm to (112.8, 59.7)
- moved J40 90.8 mm to (117.4, 59.7)
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Connections:
- J34 pad 1: unconnected-(J34-Pin_1-Pad1) -> /CloudController/Output1
- J34 pad 2: unconnected-(J34-Pin_2-Pad2) -> /CloudController/Output6
- J34 pad 3: unconnected-(J34-Pin_3-Pad3) -> /CloudController/Output11
- J34 pad 4: unconnected-(J34-Pin_4-Pad4) -> +5V
- J37 pad 1: unconnected-(J37-Pin_1-Pad1) -> /CloudController/Output2
- J37 pad 2: unconnected-(J37-Pin_2-Pad2) -> /CloudController/Output7
- J37 pad 3: unconnected-(J37-Pin_3-Pad3) -> /CloudController/Output12
- J37 pad 4: unconnected-(J37-Pin_4-Pad4) -> +5V
- J40 pad 1: unconnected-(J40-Pin_1-Pad1) -> /CloudController/Output3
- J40 pad 2: unconnected-(J40-Pin_2-Pad2) -> /CloudController/Output8
- J40 pad 3: unconnected-(J40-Pin_3-Pad3) -> /CloudController/Output13
- J40 pad 4: unconnected-(J40-Pin_4-Pad4) -> +5V
- J43 pad 1: unconnected-(J43-Pin_1-Pad1) -> /CloudController/Output4
- J43 pad 2: unconnected-(J43-Pin_2-Pad2) -> /CloudController/Output9
- J43 pad 3: unconnected-(J43-Pin_3-Pad3) -> /CloudController/Output14
- J43 pad 4: unconnected-(J43-Pin_4-Pad4) -> +5V
- J52 pad 1: unconnected-(J52-Pin_1-Pad1) -> /CloudController/Output5
- J52 pad 2: unconnected-(J52-Pin_2-Pad2) -> /CloudController/Output10
- J52 pad 3: unconnected-(J52-Pin_3-Pad3) -> /CloudController/Output15
- J52 pad 4: unconnected-(J52-Pin_4-Pad4) -> +5V
Routing:
- net /SDA: track 9.32 -> 65.6 mm, vias 0 -> 1
- net /SCL: track 12.5 -> 58.8 mm
- net /CloudController/Output14: track 0.00 -> 18.7 mm
- net /CloudController/Output11: track 0.00 -> 18.6 mm
- net /CloudController/Output1: track 0.00 -> 18.1 mm
- net /CloudController/Output4: track 0.00 -> 17.7 mm
- net /CloudController/Output13: track 0.00 -> 17.6 mm
- net /CloudController/Output15: track 0.00 -> 17.6 mm
- net /CloudController/Output9: track 0.00 -> 17.4 mm
- net /CloudController/Output6: track 0.00 -> 17.3 mm
- net /CloudController/Output3: track 0.00 -> 17.1 mm
- net /CloudController/Output5: track 0.00 -> 17.1 mm
- net /CloudController/Output2: track 0.00 -> 16.9 mm
- net /CloudController/Output12: track 0.00 -> 16.9 mm
- net /CloudController/Output8: track 0.00 -> 16.3 mm
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- added copper zone on B.Cu, net +5V

Commit message: Routing done!
Routing:
- net GND: track 0.00 -> 245.0 mm, vias 0 -> 16
- net /Control5: track 0.00 -> 121.9 mm
- net /Control6: track 0.00 -> 96.8 mm
- net /Control10: track 0.00 -> 92.5 mm, vias 0 -> 1
- net /Control15: track 0.00 -> 86.8 mm, vias 0 -> 1
- net /Control4: track 0.00 -> 85.7 mm, vias 0 -> 1
- net +5V: track 62.2 -> 146.4 mm, vias 21 -> 35
- net /Control11: track 0.00 -> 84.3 mm, vias 0 -> 1
- net /Control14: track 0.00 -> 81.4 mm, vias 0 -> 1
- net /Control12: track 0.00 -> 80.7 mm, vias 0 -> 1
- net /Control9: track 0.00 -> 75.6 mm, vias 0 -> 1
- net Net-(J25-Pin_1): track 0.00 -> 69.2 mm
- net Net-(J26-Pin_1): track 0.00 -> 68.0 mm
- net Net-(J5-Pin_1): track 0.00 -> 66.2 mm
- net /Control7: track 0.00 -> 65.3 mm
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
Commit message: Routing
Other:
- board text added: "GNCTR Cloud Star PCB Aleks Berezowski"
Changed lines of the file:
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@@
   (gr_rect (start 25 25) (end 125 125)
     (stroke (width 0.1) (type default)) (fill none) (layer "Edge.Cuts"))
+  (gr_text "GNCTR Cloud Star PCB\nAleks Berezowski" (at 42.418 40.005 90) (layer "F.SilkS")
+    (effects (font (size 1.5 1.5) (thickness 0.3) bold) (justify bottom))
+  )
   (segment (start 67.1068 71.475001) (end 65.662944 71.475001) (width 0.25) (layer "F.Cu") (net 1))
   (segment (start 60.198 51.816) (end 60.198 50.172) (width 0.25) (layer "F.Cu") (net 1))

Commit message: Routing
Connections:
- U2 pad 10: unconnected-(U2-D19/VSPI_MISO-Pad10) -> /Control15
- U2 pad 19: /Control14 -> unconnected-(U2-D34/ADC1_CH6-Pad19)
- U2 pad 20: /Control15 -> unconnected-(U2-D35/ADC1_CH7-Pad20)
- U2 pad 7: unconnected-(U2-TX2/D17-Pad7) -> /Control3
- U2 pad 8: /Control3 -> unconnected-(U2-D5/VSPI_CS0-Pad8)
- U2 pad 9: unconnected-(U2-D18/VSPI_CLK-Pad9) -> /Control14
Routing:
- net /Control14: track 81.4 -> 50.3 mm
- net /Control15: track 86.8 -> 93.0 mm, vias 1 -> 3
- net /Control3: track 43.2 -> 42.0 mm

Commit message: Finalize rev2 order
- added comments, silk screens
- exported PDF and gerber
Other:
- board text added: "3V3 GND"
- board text added: "5V GND"
- board text added: "GNCTR Cloud Star PCB Aleks Berezowski Rev2 | 2023-12-01"
- board text added: "GND 3V3"
- board text added: "GND 5V"
- board text added: "R-G-B-VCC"
- board text added: "Top: In-Line R to GPIO Bottom: Pull-Downs"
- board text removed: "GNCTR Cloud Star PCB Aleks Berezowski"
