File: Cloud-Star-Lights-PCB/CloudControlCircuit1.kicad_sch (KiCad schematic)
At the start: 3 parts, among them Q1 BS170

Commit message: Finalize rev2 order
- added comments, silk screens
- exported PDF and gerber
Parts:
- renumbered R32 to R49, R32 to R50
Other:
- note added: "FIXME: Common ground should be used; don't use hierarchical pin for GND"
- note added: "Note: The top inline resistor is largely unnecessary, and it can be shorted/0 ohm."
