File: Star-PCB/Star-PCB/Star-PCB.kicad_sch (KiCad schematic)
At the start: 6 parts

Commit message: Schematics Done
Parts:
- removed R1: ~, Resistor_SMD:R_0201_0603Metric, symbol Star-Library:ERJP03J220V
Connections:
- net at D1.1, D2.1, D3.1: now also J1.1
Changed lines of the file:
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@@
-    (stroke (width 0) (type default))
-  )
-  (wire (pts (xy 107.95 90.17) (xy 110.49 90.17))
     (stroke (width 0) (type default))
   )
@@
     (stroke (width 0) (type default))
   )
-  (wire (pts (xy 95.25 90.17) (xy 97.79 90.17))
+  (wire (pts (xy 95.25 90.17) (xy 110.49 90.17))
     (stroke (width 0) (type default))
   )
@@
         )
       )
-    )
-  )
-  (symbol (lib_id "Star-Library:ERJP03J220V") (at 102.87 90.17 0) (unit 1)
-    (in_bom yes) (on_board yes) (dnp no) (fields_autoplaced)
-    (property "Reference" "R1" (at 102.87 86.36 0)
-      (effects (font (size 1.27 1.27)))
-    )
-    (property "Value" "~" (at 102.87 90.17 0)
-      (effects (font (size 1.27 1.27)))
-    )
-    (property "Footprint" "Resistor_SMD:R_0201_0603Metric" (at 102.87 90.17 0)
-      (effects (font (size 1.27 1.27)) hide)
-    )
-    (property "Datasheet" "" (at 102.87 90.17 0)
-      (effects (font (size 1.27 1.27)) hide)
-    )
-    (pin "1")
-    (pin "2")
-    (instances
-      (project "Star-PCB"
-        (path "/89137b40-bd1a-4b6b-9428-fda32c28674d"
-          (reference "R1") (unit 1)
-        )
-      )

Commit message: Schematic Changes
Parts:
- removed J1, J2: ~, Star-Library:EST026, symbol Star-Library:EST026
- added J3: Conn_01x02, symbol Connector_Generic:Conn_01x02
Connections:
- net at D1.1, D2.1, D3.1: now also J3.2 (Pin_2)
- net at D1.2, D2.2, D3.2: now also J3.1 (Pin_1)
Changed lines of the file:
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@@
   (junction (at 130.81 91.44) (diameter 0) (color 0 0 0 0)
   )
-  (junction (at 130.81 90.17) (diameter 0) (color 0 0 0 0)
+  (junction (at 130.81 102.87) (diameter 0) (color 0 0 0 0)
   )
-  (junction (at 110.49 90.17) (diameter 0) (color 0 0 0 0)
+  (junction (at 110.49 102.87) (diameter 0) (color 0 0 0 0)
   )
   (junction (at 110.49 91.44) (diameter 0) (color 0 0 0 0)
-  )
-  (wire (pts (xy 130.81 90.17) (xy 130.81 91.44))
-    (stroke (width 0) (type default))
   )
   (wire (pts (xy 127 80.01) (xy 130.81 80.01))
     (stroke (width 0) (type default))
   )
-  (wire (pts (xy 110.49 80.01) (xy 110.49 90.17))
+  (wire (pts (xy 110.49 111.76) (xy 110.49 102.87))
     (stroke (width 0) (type default))
   )
-  (wire (pts (xy 130.81 90.17) (xy 133.35 90.17))
+  (wire (pts (xy 110.49 80.01) (xy 110.49 91.44))
     (stroke (width 0) (type default))
   )
@@
   )
   (wire (pts (xy 110.49 91.44) (xy 115.57 91.44))
-    (stroke (width 0) (type default))
-  )
-  (wire (pts (xy 110.49 90.17) (xy 110.49 91.44))
     (stroke (width 0) (type default))
   )
@@
     (stroke (width 0) (type default))
   )
+  (wire (pts (xy 119.38 111.76) (xy 110.49 111.76))
+    (stroke (width 0) (type default))
+  )
   (wire (pts (xy 115.57 102.87) (xy 110.49 102.87))
     (stroke (width 0) (type default))
@@
     (stroke (width 0) (type default))
   )
-  (wire (pts (xy 130.81 80.01) (xy 130.81 90.17))
+  (wire (pts (xy 130.81 102.87) (xy 130.81 111.76))
     (stroke (width 0) (type default))
   )
-  (wire (pts (xy 95.25 90.17) (xy 110.49 90.17))
+  (wire (pts (xy 130.81 80.01) (xy 130.81 91.44))
+    (stroke (width 0) (type default))
+  )
+  (wire (pts (xy 121.92 111.76) (xy 130.81 111.76))
     (stroke (width 0) (type default))
   )
@@
     )
   )
-  (symbol (lib_id "Star-Library:EST026") (at 95.25 86.36 0) (unit 1)
+  (symbol (lib_id "Connector_Generic:Conn_01x02") (at 121.92 116.84 270) (unit 1)
     (in_bom yes) (on_board yes) (dnp no) (fields_autoplaced)
-    (property "Reference" "J1" (at 92.71 87.63 0)
-      (effects (font (size 1.27 1.27)))
+    (property "Reference" "J3" (at 124.46 115.57 90)
+      (effects (font (size 1.27 1.27)) (justify left))
     )
-    (property "Value" "~" (at 95.25 86.36 0)
-      (effects (font (size 1.27 1.27)))
+    (property "Value" "Conn_01x02" (at 124.46 118.11 90)
+      (effects (font (size 1.27 1.27)) (justify left))
     )
-    (property "Footprint" "Star-Library:EST026" (at 95.25 86.36 0)
+    (property "Footprint" "" (at 121.92 116.84 0)
       (effects (font (size 1.27 1.27)) hide)
     )
-    (property "Datasheet" "" (at 95.25 86.36 0)
+    (property "Datasheet" "~" (at 121.92 116.84 0)
       (effects (font (size 1.27 1.27)) hide)
     )
     (pin "1")
+    (pin "2")
     (instances
       (project "Star-PCB"
         (path "/89137b40-bd1a-4b6b-9428-fda32c28674d"
-          (reference "J1") (unit 1)
+          (reference "J3") (unit 1)
         )
       )
-    )
-  )
-  (symbol (lib_id "Star-Library:EST026") (at 133.35 86.36 0) (mirror y) (unit 1)
-    (in_bom yes) (on_board yes) (dnp no)
-    (property "Reference" "J2" (at 135.89 87.63 0)
-      (effects (font (size 1.27 1.27)))
-    )
-    (property "Value" "~" (at 133.35 86.36 0)
-      (effects (font (size 1.27 1.27)))
-    )
-    (property "Footprint" "Star-Library:EST026" (at 133.35 86.36 0)
-      (effects (font (size 1.27 1.27)) hide)
-    )
-    (property "Datasheet" "" (at 133.35 86.36 0)
-      (effects (font (size 1.27 1.27)) hide)
-    )
-    (pin "1")
-    (instances
-      (project "Star-PCB"
-        (path "/89137b40-bd1a-4b6b-9428-fda32c28674d"
-          (reference "J2") (unit 1)
-        )
-      )

Commit message: DONE!
Parts:
- added H1, H2, H3, H4: MountingHole_Pad, MountingHole:MountingHole_4.3mm_M4_ISO7380_Pad_TopBottom, symbol Mechanical:MountingHole_Pad
- added J1: Conn_01x02, Star-Library:star_connector, symbol Connector_Generic:Conn_01x02
- J2: renamed from J3; footprint (none) -> Connector_PinHeader_2.54mm:PinHeader_1x02_P2.54mm_Vertical
Connections:
- net at D1.1, D2.1, D3.1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: now also J1.2 (Pin_2)
- net at D1.2, D2.2, D3.2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: now also J1.1 (Pin_1)
- no-connect marks 0 -> 4
Other:
- moved on the sheet: J2
Changed lines of the file:
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@@
   (junction (at 130.81 91.44) (diameter 0) (color 0 0 0 0)
   )
+  (junction (at 130.81 113.03) (diameter 0) (color 0 0 0 0)
+  )
   (junction (at 130.81 102.87) (diameter 0) (color 0 0 0 0)
   )
   (junction (at 110.49 102.87) (diameter 0) (color 0 0 0 0)
   )
+  (junction (at 110.49 113.03) (diameter 0) (color 0 0 0 0)
+  )
   (junction (at 110.49 91.44) (diameter 0) (color 0 0 0 0)
   )
+  (no_connect (at 66.04 68.58))
+  (no_connect (at 92.71 68.58))
+  (no_connect (at 83.82 68.58))
+  (no_connect (at 73.66 68.58))
   (wire (pts (xy 127 80.01) (xy 130.81 80.01))
     (stroke (width 0) (type default))
   )
-  (wire (pts (xy 110.49 111.76) (xy 110.49 102.87))
+  (wire (pts (xy 110.49 123.19) (xy 110.49 113.03))
     (stroke (width 0) (type default))
   )
@@
     (stroke (width 0) (type default))
   )
+  (wire (pts (xy 110.49 113.03) (xy 119.38 113.03))
+    (stroke (width 0) (type default))
+  )
   (wire (pts (xy 127 91.44) (xy 130.81 91.44))
     (stroke (width 0) (type default))
@@
     (stroke (width 0) (type default))
   )
-  (wire (pts (xy 119.38 111.76) (xy 110.49 111.76))
+  (wire (pts (xy 119.38 123.19) (xy 110.49 123.19))
+    (stroke (width 0) (type default))
+  )
+  (wire (pts (xy 130.81 113.03) (xy 130.81 123.19))
     (stroke (width 0) (type default))
   )
@@
     (stroke (width 0) (type default))
   )
-  (wire (pts (xy 130.81 102.87) (xy 130.81 111.76))
+  (wire (pts (xy 130.81 102.87) (xy 130.81 113.03))
+    (stroke (width 0) (type default))
+  )
+  (wire (pts (xy 110.49 113.03) (xy 110.49 102.87))
     (stroke (width 0) (type default))
   )
@@
     (stroke (width 0) (type default))
   )
-  (wire (pts (xy 121.92 111.76) (xy 130.81 111.76))
+  (wire (pts (xy 121.92 113.03) (xy 130.81 113.03))
+    (stroke (width 0) (type default))
+  )
+  (wire (pts (xy 121.92 123.19) (xy 130.81 123.19))
     (stroke (width 0) (type default))
   )
@@
     )
   )
-  (symbol (lib_id "Connector_Generic:Conn_01x02") (at 121.92 116.84 270) (unit 1)
-    (in_bom yes) (on_board yes) (dnp no) (fields_autoplaced)
-    (property "Reference" "J3" (at 124.46 115.57 90)
-      (effects (font (size 1.27 1.27)) (justify left))
-    )
-    (property "Value" "Conn_01x02" (at 124.46 118.11 90)
-      (effects (font (size 1.27 1.27)) (justify left))
-    )
-    (property "Footprint" "" (at 121.92 116.84 0)
-      (effects (font (size 1.27 1.27)) hide)
-    )
-    (property "Datasheet" "~" (at 121.92 116.84 0)
+  (symbol (lib_id "Connector_Generic:Conn_01x02") (at 121.92 118.11 270) (unit 1)
+    (in_bom yes) (on_board yes) (dnp no) (fields_autoplaced)
+    (property "Reference" "J1" (at 124.46 116.84 90)
+      (effects (font (size 1.27 1.27)) (justify left))
+    )
+    (property "Value" "Conn_01x02" (at 124.46 119.38 90)
+      (effects (font (size 1.27 1.27)) (justify left) hide)
+    )
+    (property "Footprint" "Star-Library:star_connector" (at 121.92 118.11 0)
+      (effects (font (size 1.27 1.27)) hide)
+    )
+    (property "Datasheet" "~" (at 121.92 118.11 0)
       (effects (font (size 1.27 1.27)) hide)
     )
@@
       (project "Star-PCB"
         (path "/89137b40-bd1a-4b6b-9428-fda32c28674d"
-          (reference "J3") (unit 1)
-        )
-      )
+          (reference "J1") (unit 1)
+        )
+      )
+    )
+  )
+  (symbol (lib_id "Mechanical:MountingHole_Pad") (at 92.71 66.04 0) (unit 1)
+    (in_bom yes) (on_board yes) (dnp no) (fields_autoplaced)
+    (property "Reference" "H4" (at 95.25 63.5 0)
+      (effects (font (size 1.27 1.27)) (justify left))
+    )
+    (property "Value" "MountingHole_Pad" (at 95.25 66.04 0)
+      (effects (font (size 1.27 1.27)) (justify left) hide)
+    )
+    (property "Footprint" "MountingHole:MountingHole_4.3mm_M4_ISO7380_Pad_TopBottom" (at 92.71 66.04 0)
+      (effects (font (size 1.27 1.27)) hide)
+    )
+    (property "Datasheet" "~" (at 92.71 66.04 0)
+      (effects (font (size 1.27 1.27)) hide)
+    )
+    (pin "1")
+    (instances
+      (project "Star-PCB"
+        (path "/89137b40-bd1a-4b6b-9428-fda32c28674d"
+          (reference "H4") (unit 1)
+        )
+      )
+    )
+  )
+  (symbol (lib_id "Connector_Generic:Conn_01x02") (at 121.92 128.27 270) (unit 1)
+    (in_bom yes) (on_board yes) (dnp no) (fields_autoplaced)
+    (property "Reference" "J2" (at 124.46 127 90)
+      (effects (font (size 1.27 1.27)) (justify left))
+    )
+    (property "Value" "Conn_01x02" (at 124.46 129.54 90)
+      (effects (font (size 1.27 1.27)) (justify left))
+    )
+    (property "Footprint" "Connector_PinHeader_2.54mm:PinHeader_1x02_P2.54mm_Vertical" (at 121.92 128.27 0)
+      (effects (font (size 1.27 1.27)) hide)
+    )
+    (property "Datasheet" "~" (at 121.92 128.27 0)
+      (effects (font (size 1.27 1.27)) hide)
+    )
+    (pin "1")
+    (pin "2")
+    (instances
+      (project "Star-PCB"
+        (path "/89137b40-bd1a-4b6b-9428-fda32c28674d"
+          (reference "J2") (unit 1)
+        )
+      )
+    )
+  )
+  (symbol (lib_id "Mechanical:MountingHole_Pad") (at 83.82 66.04 0) (unit 1)
+    (in_bom yes) (on_board yes) (dnp no) (fields_autoplaced)
+    (property "Reference" "H3" (at 86.36 63.5 0)
+      (effects (font (size 1.27 1.27)) (justify left))
+    )
+    (property "Value" "MountingHole_Pad" (at 86.36 66.04 0)
+      (effects (font (size 1.27 1.27)) (justify left) hide)
+    )
+    (property "Footprint" "MountingHole:MountingHole_4.3mm_M4_ISO7380_Pad_TopBottom" (at 83.82 66.04 0)
+      (effects (font (size 1.27 1.27)) hide)
+    )
+    (property "Datasheet" "~" (at 83.82 66.04 0)
+      (effects (font (size 1.27 1.27)) hide)
+    )
+    (pin "1")
+    (instances
+      (project "Star-PCB"
+        (path "/89137b40-bd1a-4b6b-9428-fda32c28674d"
+          (reference "H3") (unit 1)
+        )
+      )
+    )
+  )
+  (symbol (lib_id "Mechanical:MountingHole_Pad") (at 73.66 66.04 0) (unit 1)
+    (in_bom yes) (on_board yes) (dnp no) (fields_autoplaced)
+    (property "Reference" "H2" (at 76.2 63.5 0)
+      (effects (font (size 1.27 1.27)) (justify left))
+    )
+    (property "Value" "MountingHole_Pad" (at 76.2 66.04 0)
+      (effects (font (size 1.27 1.27)) (justify left) hide)
+    )
+    (property "Footprint" "MountingHole:MountingHole_4.3mm_M4_ISO7380_Pad_TopBottom" (at 73.66 66.04 0)
+      (effects (font (size 1.27 1.27)) hide)
+    )
+    (property "Datasheet" "~" (at 73.66 66.04 0)
+      (effects (font (size 1.27 1.27)) hide)
+    )
+    (pin "1")
+    (instances
+      (project "Star-PCB"
+        (path "/89137b40-bd1a-4b6b-9428-fda32c28674d"
+          (reference "H2") (unit 1)
+        )
+      )
+    )
+  )
+  (symbol (lib_id "Mechanical:MountingHole_Pad") (at 66.04 66.04 0) (unit 1)
+    (in_bom yes) (on_board yes) (dnp no) (fields_autoplaced)
+    (property "Reference" "H1" (at 68.58 63.5 0)
+      (effects (font (size 1.27 1.27)) (justify left))
+    )
+    (property "Value" "MountingHole_Pad" (at 68.58 66.04 0)
+      (effects (font (size 1.27 1.27)) (justify left) hide)
+    )
+    (property "Footprint" "MountingHole:MountingHole_4.3mm_M4_ISO7380_Pad_TopBottom" (at 66.04 66.04 0)
+      (effects (font (size 1.27 1.27)) hide)
+    )
+    (property "Datasheet" "~" (at 66.04 66.04 0)
+      (effects (font (size 1.27 1.27)) hide)
+    )
+    (pin "1")
+    (instances
+      (project "Star-PCB"
+        (path "/89137b40-bd1a-4b6b-9428-fda32c28674d"
+          (reference "H1") (unit 1)
+        )
+      )
