File: Star-PCB/Star-PCB/Star-PCB.kicad_pcb (KiCad board)
At the start: 2 copper layers, 6 parts

Commit message: Hopefully make PCB?
Parts:
- moved D1 111.8 mm to (172.0, 124.0), turned to 90 degrees
- moved D3 108.7 mm to (212.0, 35.0), turned to 90 degrees
- moved D2 52.7 mm to (127.0, 35.0), turned to 90 degrees
- moved J2 48.5 mm to (123.5, 78.0)
- moved R1 33.3 mm to (132.7, 88.0)
- moved J1 20.2 mm to (123.9, 88.0)
Connections:
- R1 pad 2: Net-(D1-Pad1) -> Net-(J1-Pad1)
Routing:
- net Net-(D1-Pad2): track 0.00 -> 8.76 mm, vias 0 -> 3
- net Net-(J1-Pad1): track 0.00 -> 3.00 mm
- net Net-(D1-Pad1): track 0.00 -> 0.51 mm
- added copper zone on F.Cu, net Net-(D1-Pad1)
- added copper zone on B.Cu, net Net-(D1-Pad2)
Other:
- board outline added: 100 x 100 mm
Changed lines of the file:
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@@
   (net 9 "Net-(J1-Pad1)")
   (footprint "Star-Library:LY_E65F-DAEA-35-3B5A-50-R33-Z" (layer "F.Cu")
-    (at 73.12 71.77)
+    (at 172 124 90)
     (property "Sheetfile" "Star-PCB.kicad_sch")
     (property "Sheetname" "")
     (attr smd)
-    (fp_text reference "D1" (at 0 -10.16 unlocked) (layer "F.SilkS")
+    (fp_text reference "D1" (at 0 -10.16 90 unlocked) (layer "F.SilkS")
         (effects (font (size 1 1) (thickness 0.1)))
     )
-    (fp_text value "~" (at 0 -8.66 unlocked) (layer "F.Fab")
+    (fp_text value "~" (at 0 -8.66 90 unlocked) (layer "F.Fab")
         (effects (font (size 1 1) (thickness 0.15)))
     )
-    (fp_text user "${REFERENCE}" (at 0 -7.16 unlocked) (layer "F.Fab")
+    (fp_text user "${REFERENCE}" (at 0 -7.16 90 unlocked) (layer "F.Fab")
         (effects (font (size 1 1) (thickness 0.15)))
     )
-    (pad "1" smd rect (at -2 -3.15) (size 3.3 4.8) (layers "F.Cu" "F.Paste" "F.Mask")
+    (pad "1" smd rect (at -2 -3.15 90) (size 3.3 4.8) (layers "F.Cu" "F.Paste" "F.Mask")
       (net 1 "Net-(D1-Pad1)") (pinfunction "1") (pintype "input") (thermal_bridge_angle 45))
-    (pad "2" smd rect (at 2 3.15) (size 3.3 4.8) (layers "F.Cu" "F.Paste" "F.Mask")
+    (pad "2" smd rect (at 2 3.15 90) (size 3.3 4.8) (layers "F.Cu" "F.Paste" "F.Mask")
       (net 2 "Net-(D1-Pad2)") (pinfunction "2") (pintype "input") (thermal_bridge_angle 45))
-    (pad "3" smd rect (at 2 -3.15) (size 3.3 4.8) (layers "F.Cu" "F.Paste" "F.Mask")
+    (pad "3" smd rect (at 2 -3.15 90) (size 3.3 4.8) (layers "F.Cu" "F.Paste" "F.Mask")
       (net 3 "unconnected-(D1-Pad3)") (pinfunction "3") (pintype "no_connect") (thermal_bridge_angle 45))
-    (pad "4" smd rect (at -2 3.15) (size 3.3 4.8) (layers "F.Cu" "F.Paste" "F.Mask")
+    (pad "4" smd rect (at -2 3.15 90) (size 3.3 4.8) (layers "F.Cu" "F.Paste" "F.Mask")
       (net 4 "unconnected-(D1-Pad4)") (pinfunction "4") (pintype "no_connect") (thermal_bridge_angle 45))
   )
   (footprint "Star-Library:LY_E65F-DAEA-35-3B5A-50-R33-Z" (layer "F.Cu")
-    (at 89.19 71.77)
+    (at 127 35 90)
     (property "Sheetfile" "Star-PCB.kicad_sch")
     (property "Sheetname" "")
     (attr smd)
-    (fp_text reference "D2" (at 0 -10.16 unlocked) (layer "F.SilkS")
+    (fp_text reference "D2" (at 0 -10.16 90 unlocked) (layer "F.SilkS")
         (effects (font (size 1 1) (thickness 0.1)))
     )
-    (fp_text value "~" (at 0 -8.66 unlocked) (layer "F.Fab")
+    (fp_text value "~" (at 0 -8.66 90 unlocked) (layer "F.Fab")
         (effects (font (size 1 1) (thickness 0.15)))
     )
-    (fp_text user "${REFERENCE}" (at 0 -7.16 unlocked) (layer "F.Fab")
+    (fp_text user "${REFERENCE}" (at 0 -7.16 90 unlocked) (layer "F.Fab")
         (effects (font (size 1 1) (thickness 0.15)))
     )
-    (pad "1" smd rect (at -2 -3.15) (size 3.3 4.8) (layers "F.Cu" "F.Paste" "F.Mask")
+    (pad "1" smd rect (at -2 -3.15 90) (size 3.3 4.8) (layers "F.Cu" "F.Paste" "F.Mask")
       (net 1 "Net-(D1-Pad1)") (pinfunction "1") (pintype "input") (thermal_bridge_angle 45))
-    (pad "2" smd rect (at 2 3.15) (size 3.3 4.8) (layers "F.Cu" "F.Paste" "F.Mask")
+    (pad "2" smd rect (at 2 3.15 90) (size 3.3 4.8) (layers "F.Cu" "F.Paste" "F.Mask")
       (net 2 "Net-(D1-Pad2)") (pinfunction "2") (pintype "input") (thermal_bridge_angle 45))
-    (pad "3" smd rect (at 2 -3.15) (size 3.3 4.8) (layers "F.Cu" "F.Paste" "F.Mask")
+    (pad "3" smd rect (at 2 -3.15 90) (size 3.3 4.8) (layers "F.Cu" "F.Paste" "F.Mask")
       (net 5 "unconnected-(D2-Pad3)") (pinfunction "3") (pintype "no_connect") (thermal_bridge_angle 45))
-    (pad "4" smd rect (at -2 3.15) (size 3.3 4.8) (layers "F.Cu" "F.Paste" "F.Mask")
+    (pad "4" smd rect (at -2 3.15 90) (size 3.3 4.8) (layers "F.Cu" "F.Paste" "F.Mask")
       (net 6 "unconnected-(D2-Pad4)") (pinfunction "4") (pintype "no_connect") (thermal_bridge_angle 45))
   )
   (footprint "Star-Library:EST026" (layer "F.Cu")
-    (at 76.2 88.9)
+    (at 123.46 78)
     (property "Sheetfile" "Star-PCB.kicad_sch")
     (property "Sheetname" "")
@@
   )
   (footprint "Star-Library:EST026" (layer "F.Cu")
-    (at 104.14 83.82)
+    (at 123.92 88)
     (property "Sheetfile" "Star-PCB.kicad_sch")
     (property "Sheetname" "")
@@
   )
   (footprint "Resistor_SMD:R_0201_0603Metric" (layer "F.Cu")
-    (at 99.405 86.36)
+    (at 132.655 88)
     (descr "Resistor SMD 0201 (0603 Metric), square (rectangular) end terminal, IPC_7351 nominal, (Body size source: https://www.vishay.com/docs/20052/crcw0201e3.pdf), generated with kicad-footprint-generator")
     (tags "resistor")
@@
       (net 9 "Net-(J1-Pad1)") (pinfunction "1") (pintype "bidirectional"))
     (pad "2" smd roundrect (at 0.32 0) (size 0.46 0.4) (layers "F.Cu" "F.Mask") (roundrect_rratio 0.25)
-      (net 1 "Net-(D1-Pad1)") (pinfunction "2") (pintype "bidirectional"))
+      (net 9 "Net-(J1-Pad1)") (pinfunction "2") (pintype "bidirectional"))
     (model "${KICAD6_3DMODEL_DIR}/Resistor_SMD.3dshapes/R_0201_0603Metric.wrl"
       (offset (xyz 0 0 0))
@@
   )
   (footprint "Star-Library:LY_E65F-DAEA-35-3B5A-50-R33-Z" (layer "F.Cu")
-    (at 109.76 71.77)
+    (at 212 35 90)
     (property "Sheetfile" "Star-PCB.kicad_sch")
     (property "Sheetname" "")
     (attr smd)
-    (fp_text reference "D3" (at 0 -10.16 unlocked) (layer "F.SilkS")
+    (fp_text reference "D3" (at 0 -10.16 90 unlocked) (layer "F.SilkS")
         (effects (font (size 1 1) (thickness 0.1)))
     )
-    (fp_text value "~" (at 0 -8.66 unlocked) (layer "F.Fab")
+    (fp_text value "~" (at 0 -8.66 90 unlocked) (layer "F.Fab")
         (effects (font (size 1 1) (thickness 0.15)))
     )
-    (fp_text user "${REFERENCE}" (at 0 -7.16 unlocked) (layer "F.Fab")
+    (fp_text user "${REFERENCE}" (at 0 -7.16 90 unlocked) (layer "F.Fab")
         (effects (font (size 1 1) (thickness 0.15)))
     )
-    (pad "1" smd rect (at -2 -3.15) (size 3.3 4.8) (layers "F.Cu" "F.Paste" "F.Mask")
+    (pad "1" smd rect (at -2 -3.15 90) (size 3.3 4.8) (layers "F.Cu" "F.Paste" "F.Mask")
       (net 1 "Net-(D1-Pad1)") (pinfunction "1") (pintype "input") (thermal_bridge_angle 45))
-    (pad "2" smd rect (at 2 3.15) (size 3.3 4.8) (layers "F.Cu" "F.Paste" "F.Mask")
+    (pad "2" smd rect (at 2 3.15 90) (size 3.3 4.8) (layers "F.Cu" "F.Paste" "F.Mask")
       (net 2 "Net-(D1-Pad2)") (pinfunction "2") (pintype "input") (thermal_bridge_angle 45))
-    (pad "3" smd rect (at 2 -3.15) (size 3.3 4.8) (layers "F.Cu" "F.Paste" "F.Mask")
+    (pad "3" smd rect (at 2 -3.15 90) (size 3.3 4.8) (layers "F.Cu" "F.Paste" "F.Mask")
       (net 7 "unconnected-(D3-Pad3)") (pinfunction "3") (pintype "no_connect") (thermal_bridge_angle 45))
-    (pad "4" smd rect (at -2 3.15) (size 3.3 4.8) (layers "F.Cu" "F.Paste" "F.Mask")
+    (pad "4" smd rect (at -2 3.15 90) (size 3.3 4.8) (layers "F.Cu" "F.Paste" "F.Mask")
       (net 8 "unconnected-(D3-Pad4)") (pinfunction "4") (pintype "no_connect") (thermal_bridge_angle 45))
   )
+  (gr_rect (start 120 29) (end 220 129)
+    (stroke (width 0.1) (type default)) (fill none) (layer "Edge.Cuts"))
+  (segment (start 168.34038 126) (end 168.85 126) (width 0.25) (layer "F.Cu") (net 1))
+  (segment (start 175.15 119.15) (end 175 119) (width 0.25) (layer "F.Cu") (net 2))
+  (segment (start 175.15 122) (end 175.15 119.15) (width 0.25) (layer "F.Cu") (net 2))
+  (segment (start 215.15 33) (end 218 33) (width 0.25) (layer "F.Cu") (net 2))
+  (segment (start 133 33) (end 130.15 33) (width 0.25) (layer "F.Cu") (net 2))
+  (via (at 175 119) (size 0.8) (drill 0.4) (layers "F.Cu" "B.Cu") (free) (net 2))
+  (via (at 218 33) (size 0.8) (drill 0.4) (layers "F.Cu" "B.Cu") (free) (net 2))
+  (via (at 133 33) (size 0.8) (drill 0.4) (layers "F.Cu" "B.Cu") (free) (net 2))
+  (segment (start 129 88) (end 132 88) (width 1) (layer "F.Cu") (net 9))
+  (zone (net 1) (net_name "Net-(D1-Pad1)") (layer "F.Cu") (hatch edge 0.5)
+    (priority 1)
+    (connect_pads (clearance 0.5))
+    (min_thickness 0.25) (filled_areas_thickness no)
+    (fill yes (thermal_gap 0.5) (thermal_bridge_width 0.5))
+    (polygon
+      (pts
+        (xy 120 29)
+        (xy 120 129)
+        (xy 220 129)
+        (xy 220 29)
+      )
+    )
+  )
+  (zone (net 2) (net_name "Net-(D1-Pad2)") (layer "B.Cu") (hatch edge 0.5)
+    (connect_pads (clearance 0.5))
+    (min_thickness 0.25) (filled_areas_thickness no)
+    (fill yes (thermal_gap 0.5) (thermal_bridge_width 0.5))
+    (polygon
+      (pts
+        (xy 220 29)
+        (xy 220 129)
+        (xy 120 129)
+        (xy 120 29)
+      )
+    )
+  )
 )

Commit message: Fixed it
Routing:
- net Net-(J1-Pad1): track 3.00 -> 8.08 mm
Changed lines of the file:
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@@
   (via (at 218 33) (size 0.8) (drill 0.4) (layers "F.Cu" "B.Cu") (free) (net 2))
   (via (at 133 33) (size 0.8) (drill 0.4) (layers "F.Cu" "B.Cu") (free) (net 2))
+  (segment (start 129 88) (end 123.92 88) (width 1) (layer "F.Cu") (net 9))
   (segment (start 129 88) (end 132 88) (width 1) (layer "F.Cu") (net 9))
   (zone (net 1) (net_name "Net-(D1-Pad1)") (layer "F.Cu") (hatch edge 0.5)

Commit message: DONE!
Parts:
- removed R1: ~, Resistor_SMD:R_0201_0603Metric
- added H1: MountingHole_Pad, MountingHole:MountingHole_4.3mm_M4_ISO7380_Pad_TopBottom, F.Cu at (129.5, 38.1)
- added H2: MountingHole_Pad, MountingHole:MountingHole_4.3mm_M4_ISO7380_Pad_TopBottom, F.Cu at (154.9, 38.1)
- added H3: MountingHole_Pad, MountingHole:MountingHole_4.3mm_M4_ISO7380_Pad_TopBottom, F.Cu at (154.9, 63.5)
- added H4: MountingHole_Pad, MountingHole:MountingHole_4.3mm_M4_ISO7380_Pad_TopBottom, F.Cu at (129.5, 63.5)
- J1: value ~ -> Conn_01x02; footprint Star-Library:EST026 -> Star-Library:star_connector
- J2: value ~ -> Conn_01x02; footprint Star-Library:EST026 -> Connector_PinHeader_2.54mm:PinHeader_1x02_P2.54mm_Vertical
- moved D1 84.9 mm to (129.0, 50.8), turned to 0 degrees
- moved D3 69.8 mm to (142.2, 38.1), turned to -90 degrees
- moved J1 34.4 mm to (141.7, 58.5)
- moved J2 31.7 mm to (139.7, 50.8), turned to 90 degrees
- moved D2 29.9 mm to (152.4, 50.8), turned to 0 degrees
Connections:
- D1 pad 1: Net-(D1-Pad1) -> Net-(J1-Pin_2)
- D1 pad 2: Net-(D1-Pad2) -> Net-(J1-Pin_1)
- D2 pad 1: Net-(D1-Pad1) -> Net-(J1-Pin_2)
- D2 pad 2: Net-(D1-Pad2) -> Net-(J1-Pin_1)
- D3 pad 1: Net-(D1-Pad1) -> Net-(J1-Pin_2)
- D3 pad 2: Net-(D1-Pad2) -> Net-(J1-Pin_1)
- J1 pad 1: Net-(J1-Pad1) -> Net-(J1-Pin_1)
- J2 pad 1: Net-(D1-Pad2) -> Net-(J1-Pin_1)
Routing:
- net Net-(J1-Pin_1): track 0.00 -> 11.1 mm, vias 0 -> 4
- net Net-(D1-Pad2): track 8.76 -> 0.00 mm, vias 3 -> 0
- net Net-(J1-Pad1): track 8.08 -> 0.00 mm
- net Net-(D1-Pad1): track 0.51 -> 0.00 mm
- added copper zone on B.Cu, net Net-(J1-Pin_1)
- added copper zone on F.Cu, net Net-(J1-Pin_2)
- removed copper zone on F.Cu, net Net-(D1-Pad1)
- removed copper zone on B.Cu, net Net-(D1-Pad2)
Other:
- board size 100 x 100 mm -> 35.6 x 35.6 mm

Commit message: DONE! (v2)
Routing:
- net Net-(J1-Pin_1): vias 4 -> 3
Other:
- board text added: "+"
- board text added: "-"
Changed lines of the file:
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@@
   (gr_rect (start 124.46 33.02) (end 160.02 68.58)
     (stroke (width 0.1) (type default)) (fill none) (layer "Edge.Cuts"))
+  (gr_text "-" (at 139.7 53.34) (layer "F.SilkS")
+    (effects (font (size 1 1) (thickness 0.15)) (justify right bottom))
+  )
+  (gr_text "+" (at 142.24 53.34) (layer "F.SilkS")
+    (effects (font (size 1 1) (thickness 0.15)) (justify left bottom))
+  )
   (segment (start 142.24 39.3081) (end 141.8169 39.7312) (width 0.25) (layer "F.Cu") (net 8))
   (segment (start 130.9015 51.2231) (end 131 51.2231) (width 0.25) (layer "F.Cu") (net 8))
@@
   (via (at 142.24 39.3081) (size 0.8) (drill 0.4) (layers "F.Cu" "B.Cu") (net 8))
   (via (at 130.4784 50.8) (size 0.8) (drill 0.4) (layers "F.Cu" "B.Cu") (net 8))
-  (via (at 218 33) (size 0.8) (drill 0.4) (layers "F.Cu" "B.Cu") (net 8))
   (zone (net 1) (net_name "Net-(J1-Pin_2)") (layer "F.Cu") (hatch edge 0.5)
     (priority 1)

Commit message: DONE! (v3)
Other:
- board text added: "GNCTR PCB Star Board"
Changed lines of the file:
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@@
+    (effects (font (size 1 1) (thickness 0.15)) (justify left bottom))
+  )
+  (gr_text "GNCTR PCB\nStar Board" (at 134.62 48.26) (layer "F.SilkS")
     (effects (font (size 1 1) (thickness 0.15)) (justify left bottom))
   )
@@
   (via (at 142.24 39.3081) (size 0.8) (drill 0.4) (layers "F.Cu" "B.Cu") (net 8))
   (via (at 130.4784 50.8) (size 0.8) (drill 0.4) (layers "F.Cu" "B.Cu") (net 8))
+  (zone (net 8) (net_name "Net-(J1-Pin_1)") (layer "F.Cu") (name "$teardrop_padvia$") (hatch edge 0.5)
+    (priority 30002)
+    (attr (teardrop (type padvia)))
+    (connect_pads yes (clearance 0))
+    (min_thickness 0.0254) (filled_areas_thickness no)
+    (fill yes (thermal_gap 0.5) (thermal_bridge_width 0.5) (island_removal_mode 1) (island_area_min 10))
+    (polygon
+      (pts
+        (xy 156.764465 54.514341)
+        (xy 156.941241 54.337565)
+        (xy 156.05 53.251284)
+        (xy 154.399293 53.949293)
+        (xy 156.05 55.288676)
+      )
+    )
+  )
+  (zone (net 8) (net_name "Net-(J1-Pin_1)") (layer "F.Cu") (name "$teardrop_padvia$") (hatch edge 0.5)
+    (priority 30000)
+    (attr (teardrop (type padvia)))
+    (connect_pads yes (clearance 0))
+    (min_thickness 0.0254) (filled_areas_thickness no)
+    (fill yes (thermal_gap 0.5) (thermal_bridge_width 0.5) (island_removal_mode 1) (island_area_min 10))
+    (polygon
+      (pts
+        (xy 141.9419 39.7312)
+        (xy 141.6919 39.7312)
+        (xy 141.49 38.766377)
+        (xy 139.09 40.101)
+        (xy 141.49 40.784685)
+      )
+    )
+  )
+  (zone (net 8) (net_name "Net-(J1-Pin_1)") (layer "F.Cu") (name "$teardrop_padvia$") (hatch edge 0.5)
+    (priority 30004)
+    (attr (teardrop (type padvia)))
+    (connect_pads yes (clearance 0))
+    (min_thickness 0.0254) (filled_areas_thickness no)
+    (fill yes (thermal_gap 0.5) (thermal_bridge_width 0.5) (island_removal_mode 1) (island_area_min 10))
+    (polygon
+      (pts
+        (xy 141.6919 39.932847)
+        (xy 141.9419 39.932847)
+        (xy 142.393073 39.677652)
+        (xy 142.24 39.3071)
+        (xy 141.870448 39.155027)
+      )
+    )
+  )
   (zone (net 1) (net_name "Net-(J1-Pin_2)") (layer "F.Cu") (hatch edge 0.5)
     (priority 1)
@@
       )
     )
+  )
+  (zone (net 8) (net_name "Net-(J1-Pin_1)") (layer "F.Cu") (name "$teardrop_padvia$") (hatch edge 0.5)
+    (priority 30003)
+    (attr (teardrop (type padvia)))
+    (connect_pads yes (clearance 0))
+    (min_thickness 0.0254) (filled_areas_thickness no)
+    (fill yes (thermal_gap 0.5) (thermal_bridge_width 0.5) (island_removal_mode 1) (island_area_min 10))
+    (polygon
+      (pts
+        (xy 157.2786 54.6481)
+        (xy 157.2786 54.8981)
+        (xy 157.925527 55.142652)
+        (xy 158.0796 54.7731)
+        (xy 157.925527 54.403548)
+      )
+    )
+  )
+  (zone (net 8) (net_name "Net-(J1-Pin_1)") (layer "F.Cu") (name "$teardrop_padvia$") (hatch edge 0.5)
+    (priority 30001)
+    (attr (teardrop (type padvia)))
+    (connect_pads yes (clearance 0))
+    (min_thickness 0.0254) (filled_areas_thickness no)
+    (fill yes (thermal_gap 0.5) (thermal_bridge_width 0.5) (island_removal_mode 1) (island_area_min 10))
+    (polygon
+      (pts
+        (xy 130.9015 51.0981)
+        (xy 130.9015 51.3481)
+        (xy 129.912763 51.55)
+        (xy 131.001 53.95)
+        (xy 131.914094 51.55)
+      )
+    )
+  )
+  (zone (net 8) (net_name "Net-(J1-Pin_1)") (layer "F.Cu") (name "$teardrop_padvia$") (hatch edge 0.5)
+    (priority 30005)
+    (attr (teardrop (type padvia)))
+    (connect_pads yes (clearance 0))
+    (min_thickness 0.0254) (filled_areas_thickness no)
+    (fill yes (thermal_gap 0.5) (thermal_bridge_width 0.5) (island_removal_mode 1) (island_area_min 10))
+    (polygon
+      (pts
+        (xy 131 51.3481)
+        (xy 131 51.0981)
+        (xy 130.847952 50.646927)
+        (xy 130.4774 50.8)
+        (xy 130.325327 51.169552)
+      )
+    )
